File: DSP320C6748_DVK/Mislleneous.kicad_sch (KiCad schematic)
At the start: 45 parts, among them IC17 MUN5211DW1T1G, IC18 MUN5211DW1T1G, SW1 SW_DIP_x08

Commit message: Whole Schematic Reannotation Done
Parts:
- renumbered R101 to R225, R100 to R226, R99 to R227, R98 to R228, R102 to R229, R103 to R230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
