File: DSP320C6748_DVK/NAND_Flash.kicad_sch (KiCad schematic)
At the start: 0 parts

Commit message: NAND Flash circuit and Power Testpoints added
Parts:
- added C200, C201: 0.1uF/16V/X7R, symbol Device:C_Small
- added C202: 0.01uF/16V/X7R, symbol Device:C_Small
- added C203: 1uF/10V/X5R, symbol Device:C_Small
- added FB14: MMZ2012S121A, symbol Device:FerriteBead_Small
- added R261, R262: 4.7K,5%,1/16W, symbol Device:R_Small
- added U10: (no value), symbol NAND_Flash:S34ML02G204BHI010
Connections:
- new net: R261.2, U10.C3 (~{WP})
- new net +3V3A_Flash: C200.2, C201.2, C202.2, C203.2, FB14.2, R261.1, R262.1, U10.D3 (VCC), U10.G4 (VCC), U10.H8 (VCC), U10.J6 (VCC)
- new net +3V3D: FB14.1
- new net EMA_A_1: U10.C4 (ALE)
- new net EMA_A_2: U10.D5 (CLE)
- new net EMA_D_{0}: U10.H4 (IO0)
- new net EMA_D_{10}: U10.H5 (IO10)
- new net EMA_D_{11}: U10.J15 (IO11)
- new net EMA_D_{12}: U10.H6 (IO12)
- new net EMA_D_{13}: U10.G6 (IO13)
- new net EMA_D_{14}: U10.H7 (IO14)
- new net EMA_D_{15}: U10.G7 (IO15)
- new net EMA_D_{1}: U10.J4 (IO1)
- new net EMA_D_{2}: U10.K4 (IO2)
- new net EMA_D_{3}: U10.K5 (IO3)
- new net EMA_D_{4}: U10.K6 (IO4)
- new net EMA_D_{5}: U10.J7 (IO5)
- new net EMA_D_{6}: U10.K7 (IO6)
- new net EMA_D_{7}: U10.J8 (IO7)
- new net EMA_D_{8}: U10.H3 (IO8)
- new net EMA_D_{9}: U10.J3 (IO9)
- new net EMA_WAIT_{0}: R262.2, U10.C8 (~{RB})
- new net EMA_~{CS}_{3]: U10.C6 (~{CE})
- new net EMA_~{OE}: U10.D4 (~{RE})
- new net EMA_~{WE}: U10.C7 (~{WE})
- new net GND: C200.1, C201.1, C202.1, C203.1, U10.C5 (VSS), U10.F7 (VSS), U10.K3 (VSS), U10.K8 (VSS)
Other:
- note added: "De-Cap"
- note added: "Note: All De-caps should be place within 1CM from each pin"

Commit message: Whole Schematic Reannotation Done
Parts:
- renumbered C200 to C140, C201 to C141, C202 to C142, C203 to C143, FB14 to FB7, R261 to R151, R262 to R152, U10 to U8
Changed lines of the file:
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@@
 		(in_pos_files yes)
 		(dnp no)
-		(property "Reference" "C201"
+		(property "Reference" "C141"
 			(at 55.372 46.99 90)
 			(show_name no)
@@
 			(project "DSP320C6748_DVK"
 				(path "/3a70ffc0-9fe7-4a5b-b3c2-23140355df82/60352f1f-737b-4a7c-a5ba-03bf3caf1bef"
-					(reference "C201")
+					(reference "C141")
 					(unit 1)
 				)
@@
 		(in_pos_files yes)
 		(dnp no)
-		(property "Reference" "C202"
+		(property "Reference" "C142"
 			(at 62.992 46.99 90)
 			(show_name no)
@@
 			(project "DSP320C6748_DVK"
 				(path "/3a70ffc0-9fe7-4a5b-b3c2-23140355df82/60352f1f-737b-4a7c-a5ba-03bf3caf1bef"
-					(reference "C202")
+					(reference "C142")
 					(unit 1)
 				)
@@
 		(in_pos_files yes)
 		(dnp no)
-		(property "Reference" "#PWR0366"
+		(property "Reference" "#PWR0250"
 			(at 26.67 36.83 0)
 			(hide yes)
@@
 			(project "DSP320C6748_DVK"
 				(path "/3a70ffc0-9fe7-4a5b-b3c2-23140355df82/60352f1f-737b-4a7c-a5ba-03bf3caf1bef"
-					(reference "#PWR0366")
+					(reference "#PWR0250")
 					(unit 1)
 				)
@@
 		(in_pos_files yes)
 		(dnp no)
-		(property "Reference" "#PWR0369"
+		(property "Reference" "#PWR0254"
 			(at 168.91 31.75 0)
 			(hide yes)
@@
 			(project "DSP320C6748_DVK"
 				(path "/3a70ffc0-9fe7-4a5b-b3c2-23140355df82/60352f1f-737b-4a7c-a5ba-03bf3caf1bef"
-					(reference "#PWR0369")
+					(reference "#PWR0254")
 					(unit 1)
 				)
@@
 		(in_pos_files yes)
 		(dnp no)
-		(property "Reference" "R261"
+		(property "Reference" "R151"
 			(at 165.1 42.164 90)
 			(show_name no)
@@
 			(project "DSP320C6748_DVK"
 				(path "/3a70ffc0-9fe7-4a5b-b3c2-23140355df82/60352f1f-737b-4a7c-a5ba-03bf3caf1bef"
-					(reference "R261")
+					(reference "R151")
 					(unit 1)
 				)
@@
 		(in_pos_files yes)
 		(dnp no)
-		(property "Reference" "#PWR0371"
+		(property "Reference" "#PWR0256"
 			(at 212.09 43.18 0)
 			(hide yes)
@@
 			(project "DSP320C6748_DVK"
 				(path "/3a70ffc0-9fe7-4a5b-b3c2-23140355df82/60352f1f-737b-4a7c-a5ba-03bf3caf1bef"
-					(reference "#PWR0371")
+					(reference "#PWR0256")
 					(unit 1)
 				)
@@
 		(in_pos_files yes)
 		(dnp no)
-		(property "Reference" "#PWR0370"
+		(property "Reference" "#PWR0255"
 			(at 179.07 43.18 0)
 			(hide yes)
@@
 			(project "DSP320C6748_DVK"
 				(path "/3a70ffc0-9fe7-4a5b-b3c2-23140355df82/60352f1f-737b-4a7c-a5ba-03bf3caf1bef"
-					(reference "#PWR0370")
+					(reference "#PWR0255")
 					(unit 1)
 				)
@@
 		(in_pos_files yes)
 		(dnp no)
-		(property "Reference" "#PWR0368"
+		(property "Reference" "#PWR0251"
 			(at 45.72 62.23 0)
 			(hide yes)
@@
 			(project "DSP320C6748_DVK"
 				(path "/3a70ffc0-9fe7-4a5b-b3c2-23140355df82/60352f1f-737b-4a7c-a5ba-03bf3caf1bef"
-					(reference "#PWR0368")
+					(reference "#PWR0251")
 					(unit 1)
 				)
@@
 		(in_pos_files yes)
 		(dnp no)
-		(property "Reference" "C203"
+		(property "Reference" "C143"
 			(at 70.612 46.99 90)
 			(show_name no)
@@
 			(project "DSP320C6748_DVK"
 				(path "/3a70ffc0-9fe7-4a5b-b3c2-23140355df82/60352f1f-737b-4a7c-a5ba-03bf3caf1bef"
-					(reference "C203")
+					(reference "C143")
 					(unit 1)
 				)
@@
 		(in_pos_files yes)
 		(dnp no)
-		(property "Reference" "#PWR0365"
+		(property "Reference" "#PWR0252"
 			(at 68.58 36.83 0)
 			(hide yes)
@@
 			(project "DSP320C6748_DVK"
 				(path "/3a70ffc0-9fe7-4a5b-b3c2-23140355df82/60352f1f-737b-4a7c-a5ba-03bf3caf1bef"
-					(reference "#PWR0365")
+					(reference "#PWR0252")
 					(unit 1)
 				)
@@
 		(dnp no)
 		(fields_autoplaced yes)
-		(property "Reference" "U10"
+		(property "Reference" "U8"
 			(at 148.59 21.59 0)
 			(show_name no)
@@
 			(project "DSP320C6748_DVK"
 				(path "/3a70ffc0-9fe7-4a5b-b3c2-23140355df82/60352f1f-737b-4a7c-a5ba-03bf3caf1bef"
-					(reference "U10")
+					(reference "U8")
 					(unit 1)
 				)
@@
 		(in_pos_files yes)
 		(dnp no)
-		(property "Reference" "#PWR0367"
+		(property "Reference" "#PWR0253"
 			(at 129.54 27.94 0)
 			(hide yes)
@@
 			(project "DSP320C6748_DVK"
 				(path "/3a70ffc0-9fe7-4a5b-b3c2-23140355df82/60352f1f-737b-4a7c-a5ba-03bf3caf1bef"
-					(reference "#PWR0367")
+					(reference "#PWR0253")
 					(unit 1)
 				)
@@
 		(in_pos_files yes)
 		(dnp no)
-		(property "Reference" "R262"
+		(property "Reference" "R152"
 			(at 213.868 48.768 90)
 			(show_name no)
@@
 			(project "DSP320C6748_DVK"
 				(path "/3a70ffc0-9fe7-4a5b-b3c2-23140355df82/60352f1f-737b-4a7c-a5ba-03bf3caf1bef"
-					(reference "R262")
+					(reference "R152")
 					(unit 1)
 				)
@@
 		(dnp no)
 		(fields_autoplaced yes)
-		(property "Reference" "FB14"
+		(property "Reference" "FB7"
 			(at 36.7919 31.75 90)
 			(show_name no)
@@
 			(project "DSP320C6748_DVK"
 				(path "/3a70ffc0-9fe7-4a5b-b3c2-23140355df82/60352f1f-737b-4a7c-a5ba-03bf3caf1bef"
-					(reference "FB14")
+					(reference "FB7")
 					(unit 1)
 				)
@@
 		(in_pos_files yes)
 		(dnp no)
-		(property "Reference" "C200"
+		(property "Reference" "C140"
 			(at 47.752 46.99 90)
 			(show_name no)
@@
 			(project "DSP320C6748_DVK"
 				(path "/3a70ffc0-9fe7-4a5b-b3c2-23140355df82/60352f1f-737b-4a7c-a5ba-03bf3caf1bef"
-					(reference "C200")
-					(unit 1)
-				)
+					(reference "C140")
+					(unit 1)
+				)
