File: DSP320C6748_DVK/NAND_Flash.kicad_sch (KiCad schematic)
At the start: 8 parts

Commit message: Schematic Corrections-II Done
Parts:
- U8: value (none) -> S34ML02G204BHI010
Changed lines of the file:
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@@
 		(in_pos_files yes)
 		(dnp no)
-		(fields_autoplaced yes)
 		(property "Reference" "U8"
 			(at 148.59 21.59 0)
@@
 			)
 		)
-		(property "Value" ""
-			(at 148.59 68.58 0)
+		(property "Value" "S34ML02G204BHI010"
+			(at 148.336 114.554 0)
 			(show_name no)
 			(do_not_autoplace no)

Commit message: DC jack Replaced With Type-C, ADC and RTC section added
Parts:
- renumbered C140 to C142, C141 to C143, C142 to C144, C143 to C145, FB7 to FB9, R151 to R152, R152 to R153
Changed lines of the file:
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@@
 		(in_pos_files yes)
 		(dnp no)
-		(property "Reference" "C141"
+		(property "Reference" "C143"
 			(at 55.372 46.99 90)
 			(show_name no)
@@
 			(project "DSP320C6748_DVK"
 				(path "/3a70ffc0-9fe7-4a5b-b3c2-23140355df82/60352f1f-737b-4a7c-a5ba-03bf3caf1bef"
-					(reference "C141")
+					(reference "C143")
 					(unit 1)
 				)
@@
 		(in_pos_files yes)
 		(dnp no)
-		(property "Reference" "C142"
+		(property "Reference" "C144"
 			(at 62.992 46.99 90)
 			(show_name no)
@@
 			(project "DSP320C6748_DVK"
 				(path "/3a70ffc0-9fe7-4a5b-b3c2-23140355df82/60352f1f-737b-4a7c-a5ba-03bf3caf1bef"
-					(reference "C142")
+					(reference "C144")
 					(unit 1)
 				)
@@
 		(in_pos_files yes)
 		(dnp no)
-		(property "Reference" "#PWR0250"
+		(property "Reference" "#PWR0261"
 			(at 26.67 36.83 0)
 			(hide yes)
@@
 			(project "DSP320C6748_DVK"
 				(path "/3a70ffc0-9fe7-4a5b-b3c2-23140355df82/60352f1f-737b-4a7c-a5ba-03bf3caf1bef"
-					(reference "#PWR0250")
+					(reference "#PWR0261")
 					(unit 1)
 				)
@@
 		(in_pos_files yes)
 		(dnp no)
-		(property "Reference" "#PWR0254"
+		(property "Reference" "#PWR0265"
 			(at 168.91 31.75 0)
 			(hide yes)
@@
 			(project "DSP320C6748_DVK"
 				(path "/3a70ffc0-9fe7-4a5b-b3c2-23140355df82/60352f1f-737b-4a7c-a5ba-03bf3caf1bef"
-					(reference "#PWR0254")
+					(reference "#PWR0265")
 					(unit 1)
 				)
@@
 		(in_pos_files yes)
 		(dnp no)
-		(property "Reference" "R151"
+		(property "Reference" "R152"
 			(at 165.1 42.164 90)
 			(show_name no)
@@
 			(project "DSP320C6748_DVK"
 				(path "/3a70ffc0-9fe7-4a5b-b3c2-23140355df82/60352f1f-737b-4a7c-a5ba-03bf3caf1bef"
-					(reference "R151")
+					(reference "R152")
 					(unit 1)
 				)
@@
 		(in_pos_files yes)
 		(dnp no)
-		(property "Reference" "#PWR0256"
+		(property "Reference" "#PWR0267"
 			(at 212.09 43.18 0)
 			(hide yes)
@@
 			(project "DSP320C6748_DVK"
 				(path "/3a70ffc0-9fe7-4a5b-b3c2-23140355df82/60352f1f-737b-4a7c-a5ba-03bf3caf1bef"
-					(reference "#PWR0256")
+					(reference "#PWR0267")
 					(unit 1)
 				)
@@
 		(in_pos_files yes)
 		(dnp no)
-		(property "Reference" "#PWR0255"
+		(property "Reference" "#PWR0266"
 			(at 179.07 43.18 0)
 			(hide yes)
@@
 			(project "DSP320C6748_DVK"
 				(path "/3a70ffc0-9fe7-4a5b-b3c2-23140355df82/60352f1f-737b-4a7c-a5ba-03bf3caf1bef"
-					(reference "#PWR0255")
+					(reference "#PWR0266")
 					(unit 1)
 				)
@@
 		(dnp no)
 		(fields_autoplaced yes)
-		(property "Reference" "#G15"
+		(property "Reference" "#G11"
 			(at 260.35 166.755 0)
 			(hide yes)
@@
 			(project "DSP320C6748_DVK"
 				(path "/3a70ffc0-9fe7-4a5b-b3c2-23140355df82/60352f1f-737b-4a7c-a5ba-03bf3caf1bef"
-					(reference "#G15")
+					(reference "#G11")
 					(unit 1)
 				)
@@
 		(in_pos_files yes)
 		(dnp no)
-		(property "Reference" "#PWR0251"
+		(property "Reference" "#PWR0262"
 			(at 45.72 62.23 0)
 			(hide yes)
@@
 			(project "DSP320C6748_DVK"
 				(path "/3a70ffc0-9fe7-4a5b-b3c2-23140355df82/60352f1f-737b-4a7c-a5ba-03bf3caf1bef"
-					(reference "#PWR0251")
+					(reference "#PWR0262")
 					(unit 1)
 				)
@@
 		(in_pos_files yes)
 		(dnp no)
-		(property "Reference" "C143"
+		(property "Reference" "C145"
 			(at 70.612 46.99 90)
 			(show_name no)
@@
 			(project "DSP320C6748_DVK"
 				(path "/3a70ffc0-9fe7-4a5b-b3c2-23140355df82/60352f1f-737b-4a7c-a5ba-03bf3caf1bef"
-					(reference "C143")
+					(reference "C145")
 					(unit 1)
 				)
@@
 		(in_pos_files yes)
 		(dnp no)
-		(property "Reference" "#PWR0252"
+		(property "Reference" "#PWR0263"
 			(at 68.58 36.83 0)
 			(hide yes)
@@
 			(project "DSP320C6748_DVK"
 				(path "/3a70ffc0-9fe7-4a5b-b3c2-23140355df82/60352f1f-737b-4a7c-a5ba-03bf3caf1bef"
-					(reference "#PWR0252")
+					(reference "#PWR0263")
 					(unit 1)
 				)
@@
 		(in_pos_files yes)
 		(dnp no)
-		(property "Reference" "#PWR0253"
+		(property "Reference" "#PWR0264"
 			(at 129.54 27.94 0)
 			(hide yes)
@@
 			(project "DSP320C6748_DVK"
 				(path "/3a70ffc0-9fe7-4a5b-b3c2-23140355df82/60352f1f-737b-4a7c-a5ba-03bf3caf1bef"
-					(reference "#PWR0253")
+					(reference "#PWR0264")
 					(unit 1)
 				)
@@
 		(in_pos_files yes)
 		(dnp no)
-		(property "Reference" "R152"
+		(property "Reference" "R153"
 			(at 213.868 48.768 90)
 			(show_name no)
@@
 			(project "DSP320C6748_DVK"
 				(path "/3a70ffc0-9fe7-4a5b-b3c2-23140355df82/60352f1f-737b-4a7c-a5ba-03bf3caf1bef"
-					(reference "R152")
+					(reference "R153")
 					(unit 1)
 				)
@@
 		(dnp no)
 		(fields_autoplaced yes)
-		(property "Reference" "FB7"
+		(property "Reference" "FB9"
 			(at 36.7919 31.75 90)
 			(show_name no)
@@
 			(project "DSP320C6748_DVK"
 				(path "/3a70ffc0-9fe7-4a5b-b3c2-23140355df82/60352f1f-737b-4a7c-a5ba-03bf3caf1bef"
-					(reference "FB7")
+					(reference "FB9")
 					(unit 1)
 				)
@@
 		(in_pos_files yes)
 		(dnp no)
-		(property "Reference" "C140"
+		(property "Reference" "C142"
 			(at 47.752 46.99 90)
 			(show_name no)
@@
 			(project "DSP320C6748_DVK"
 				(path "/3a70ffc0-9fe7-4a5b-b3c2-23140355df82/60352f1f-737b-4a7c-a5ba-03bf3caf1bef"
-					(reference "C140")
-					(unit 1)
-				)
+					(reference "C142")
+					(unit 1)
+				)

Commit message: Scheamtic Re-annotation done, Some footprints assigned
Parts:
- C145: renamed from C142; footprint (none) -> Capacitor_SMD:C_0603_1608Metric_Pad1.08x0.95mm_HandSolder
- C146: renamed from C143; footprint (none) -> Capacitor_SMD:C_0603_1608Metric_Pad1.08x0.95mm_HandSolder
- C147: renamed from C144; footprint (none) -> Capacitor_SMD:C_0603_1608Metric_Pad1.08x0.95mm_HandSolder
- C148: renamed from C145; footprint (none) -> Capacitor_SMD:C_0603_1608Metric_Pad1.08x0.95mm_HandSolder
- FB10: renamed from FB9; footprint (none) -> Inductor_SMD:L_0805_2012Metric_Pad1.05x1.20mm_HandSolder
- R154: renamed from R152; footprint (none) -> Resistor_SMD:R_0603_1608Metric_Pad0.98x0.95mm_HandSolder
- R155: renamed from R153; footprint (none) -> Resistor_SMD:R_0603_1608Metric_Pad0.98x0.95mm_HandSolder
Changed lines of the file:
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@@
 		(in_pos_files yes)
 		(dnp no)
-		(property "Reference" "C143"
+		(property "Reference" "C146"
 			(at 55.372 46.99 90)
 			(show_name no)
@@
 			)
 		)
-		(property "Footprint" ""
+		(property "Footprint" "Capacitor_SMD:C_0603_1608Metric_Pad1.08x0.95mm_HandSolder"
 			(at 53.34 45.72 0)
 			(hide yes)
@@
 			(project "DSP320C6748_DVK"
 				(path "/3a70ffc0-9fe7-4a5b-b3c2-23140355df82/60352f1f-737b-4a7c-a5ba-03bf3caf1bef"
-					(reference "C143")
+					(reference "C146")
 					(unit 1)
 				)
@@
 		(in_pos_files yes)
 		(dnp no)
-		(property "Reference" "C144"
+		(property "Reference" "C147"
 			(at 62.992 46.99 90)
 			(show_name no)
@@
 			)
 		)
-		(property "Footprint" ""
+		(property "Footprint" "Capacitor_SMD:C_0603_1608Metric_Pad1.08x0.95mm_HandSolder"
 			(at 60.96 45.72 0)
 			(hide yes)
@@
 			(project "DSP320C6748_DVK"
 				(path "/3a70ffc0-9fe7-4a5b-b3c2-23140355df82/60352f1f-737b-4a7c-a5ba-03bf3caf1bef"
-					(reference "C144")
+					(reference "C147")
 					(unit 1)
 				)
@@
 		(in_pos_files yes)
 		(dnp no)
-		(property "Reference" "#PWR0261"
+		(property "Reference" "#PWR0265"
 			(at 26.67 36.83 0)
 			(hide yes)
@@
 			(project "DSP320C6748_DVK"
 				(path "/3a70ffc0-9fe7-4a5b-b3c2-23140355df82/60352f1f-737b-4a7c-a5ba-03bf3caf1bef"
-					(reference "#PWR0261")
+					(reference "#PWR0265")
 					(unit 1)
 				)
@@
 		(in_pos_files yes)
 		(dnp no)
-		(property "Reference" "#PWR0265"
+		(property "Reference" "#PWR0269"
 			(at 168.91 31.75 0)
 			(hide yes)
@@
 			(project "DSP320C6748_DVK"
 				(path "/3a70ffc0-9fe7-4a5b-b3c2-23140355df82/60352f1f-737b-4a7c-a5ba-03bf3caf1bef"
-					(reference "#PWR0265")
+					(reference "#PWR0269")
 					(unit 1)
 				)
@@
 		(in_pos_files yes)
 		(dnp no)
-		(property "Reference" "R152"
+		(property "Reference" "R154"
 			(at 165.1 42.164 90)
 			(show_name no)
@@
 			)
 		)
-		(property "Footprint" ""
+		(property "Footprint" "Resistor_SMD:R_0603_1608Metric_Pad0.98x0.95mm_HandSolder"
 			(at 171.45 43.18 0)
 			(hide yes)
@@
 			(project "DSP320C6748_DVK"
 				(path "/3a70ffc0-9fe7-4a5b-b3c2-23140355df82/60352f1f-737b-4a7c-a5ba-03bf3caf1bef"
-					(reference "R152")
+					(reference "R154")
 					(unit 1)
 				)
@@
 		(in_pos_files yes)
 		(dnp no)
-		(property "Reference" "#PWR0267"
+		(property "Reference" "#PWR0271"
 			(at 212.09 43.18 0)
 			(hide yes)
@@
 			(project "DSP320C6748_DVK"
 				(path "/3a70ffc0-9fe7-4a5b-b3c2-23140355df82/60352f1f-737b-4a7c-a5ba-03bf3caf1bef"
-					(reference "#PWR0267")
+					(reference "#PWR0271")
 					(unit 1)
 				)
@@
 		(in_pos_files yes)
 		(dnp no)
-		(property "Reference" "#PWR0266"
+		(property "Reference" "#PWR0270"
 			(at 179.07 43.18 0)
 			(hide yes)
@@
 			(project "DSP320C6748_DVK"
 				(path "/3a70ffc0-9fe7-4a5b-b3c2-23140355df82/60352f1f-737b-4a7c-a5ba-03bf3caf1bef"
-					(reference "#PWR0266")
+					(reference "#PWR0270")
 					(unit 1)
 				)
@@
 		(in_pos_files yes)
 		(dnp no)
-		(property "Reference" "#PWR0262"
+		(property "Reference" "#PWR0266"
 			(at 45.72 62.23 0)
 			(hide yes)
@@
 			(project "DSP320C6748_DVK"
 				(path "/3a70ffc0-9fe7-4a5b-b3c2-23140355df82/60352f1f-737b-4a7c-a5ba-03bf3caf1bef"
-					(reference "#PWR0262")
+					(reference "#PWR0266")
 					(unit 1)
 				)
@@
 		(in_pos_files yes)
 		(dnp no)
-		(property "Reference" "C145"
+		(property "Reference" "C148"
 			(at 70.612 46.99 90)
 			(show_name no)
@@
 			)
 		)
-		(property "Footprint" ""
+		(property "Footprint" "Capacitor_SMD:C_0603_1608Metric_Pad1.08x0.95mm_HandSolder"
 			(at 68.58 45.72 0)
 			(hide yes)
@@
 			(project "DSP320C6748_DVK"
 				(path "/3a70ffc0-9fe7-4a5b-b3c2-23140355df82/60352f1f-737b-4a7c-a5ba-03bf3caf1bef"
-					(reference "C145")
+					(reference "C148")
 					(unit 1)
 				)
@@
 		(in_pos_files yes)
 		(dnp no)
-		(property "Reference" "#PWR0263"
+		(property "Reference" "#PWR0267"
 			(at 68.58 36.83 0)
 			(hide yes)
@@
 			(project "DSP320C6748_DVK"
 				(path "/3a70ffc0-9fe7-4a5b-b3c2-23140355df82/60352f1f-737b-4a7c-a5ba-03bf3caf1bef"
-					(reference "#PWR0263")
+					(reference "#PWR0267")
 					(unit 1)
 				)
@@
 		(in_pos_files yes)
 		(dnp no)
-		(property "Reference" "#PWR0264"
+		(property "Reference" "#PWR0268"
 			(at 129.54 27.94 0)
 			(hide yes)
@@
 			(project "DSP320C6748_DVK"
 				(path "/3a70ffc0-9fe7-4a5b-b3c2-23140355df82/60352f1f-737b-4a7c-a5ba-03bf3caf1bef"
-					(reference "#PWR0264")
+					(reference "#PWR0268")
 					(unit 1)
 				)
@@
 		(in_pos_files yes)
 		(dnp no)
-		(property "Reference" "R153"
+		(property "Reference" "R155"
 			(at 213.868 48.768 90)
 			(show_name no)
@@
 			)
 		)
-		(property "Footprint" ""
+		(property "Footprint" "Resistor_SMD:R_0603_1608Metric_Pad0.98x0.95mm_HandSolder"
 			(at 212.09 46.99 0)
 			(hide yes)
@@
 			(project "DSP320C6748_DVK"
 				(path "/3a70ffc0-9fe7-4a5b-b3c2-23140355df82/60352f1f-737b-4a7c-a5ba-03bf3caf1bef"
-					(reference "R153")
+					(reference "R155")
 					(unit 1)
 				)
@@
 		(dnp no)
 		(fields_autoplaced yes)
-		(property "Reference" "FB9"
+		(property "Reference" "FB10"
 			(at 36.7919 31.75 90)
 			(show_name no)
@@
 			)
 		)
-		(property "Footprint" ""
+		(property "Footprint" "Inductor_SMD:L_0805_2012Metric_Pad1.05x1.20mm_HandSolder"
 			(at 36.83 39.878 90)
 			(hide yes)
@@
 			(project "DSP320C6748_DVK"
 				(path "/3a70ffc0-9fe7-4a5b-b3c2-23140355df82/60352f1f-737b-4a7c-a5ba-03bf3caf1bef"
-					(reference "FB9")
+					(reference "FB10")
 					(unit 1)
 				)
@@
 		(in_pos_files yes)
 		(dnp no)
-		(property "Reference" "C142"
+		(property "Reference" "C145"
 			(at 47.752 46.99 90)
 			(show_name no)
@@
 			)
 		)
-		(property "Footprint" ""
+		(property "Footprint" "Capacitor_SMD:C_0603_1608Metric_Pad1.08x0.95mm_HandSolder"
 			(at 45.72 45.72 0)
 			(hide yes)
@@
 			(project "DSP320C6748_DVK"
 				(path "/3a70ffc0-9fe7-4a5b-b3c2-23140355df82/60352f1f-737b-4a7c-a5ba-03bf3caf1bef"
-					(reference "C142")
-					(unit 1)
-				)
+					(reference "C145")
+					(unit 1)
+				)
