File: DSP320C6748_DVK/ADC_RTC.kicad_sch (KiCad schematic)
At the start: 28 parts, among them J25 POT, J26 LDR, J27 LM-35, J3 ADC_IN, U11 ADS1115IDGS, U12 LM35-LP, U13 DS1307Z+, U14 TXS0102DCU, Y7 32.768KHz

Commit message: Scheamtic Re-annotation done, Some footprints assigned
Parts:
- C208: renamed from C214; footprint (none) -> Capacitor_SMD:C_0603_1608Metric_Pad1.08x0.95mm_HandSolder
- C209: renamed from C215; footprint (none) -> Capacitor_SMD:C_0603_1608Metric_Pad1.08x0.95mm_HandSolder
- C210: renamed from C212; footprint (none) -> Capacitor_SMD:C_0603_1608Metric_Pad1.08x0.95mm_HandSolder
- C211: renamed from C205; footprint (none) -> Capacitor_SMD:C_0603_1608Metric_Pad1.08x0.95mm_HandSolder
- C212: renamed from C213; footprint (none) -> Capacitor_SMD:C_0603_1608Metric_Pad1.08x0.95mm_HandSolder
- C213: renamed from C209; footprint (none) -> Capacitor_SMD:C_0603_1608Metric_Pad1.08x0.95mm_HandSolder
- C214: renamed from C210; footprint (none) -> Capacitor_SMD:C_0603_1608Metric_Pad1.08x0.95mm_HandSolder
- C215: renamed from C211; footprint (none) -> Capacitor_SMD:C_0603_1608Metric_Pad1.08x0.95mm_HandSolder
- FB18, FB19: footprint (none) -> Inductor_SMD:L_0805_2012Metric_Pad1.05x1.20mm_HandSolder
- R270: renamed from R272; footprint (none) -> Resistor_SMD:R_0603_1608Metric_Pad0.98x0.95mm_HandSolder
- R271: renamed from R273; footprint (none) -> Resistor_SMD:R_0603_1608Metric_Pad0.98x0.95mm_HandSolder
- R272: renamed from R274; footprint (none) -> Resistor_SMD:R_0603_1608Metric_Pad0.98x0.95mm_HandSolder
- R273: renamed from R269; footprint (none) -> Resistor_SMD:R_0603_1608Metric_Pad0.98x0.95mm_HandSolder
- R274: renamed from R270; footprint (none) -> Resistor_SMD:R_0603_1608Metric_Pad0.98x0.95mm_HandSolder
- TP19: footprint (none) -> TestPoint:TestPoint_Pad_D3.0mm
- renumbered J3 to J24, R271 to R269, U12 to U11, U13 to U12, U14 to U13, U11 to U14
