File: DSP320C6748_DVK/SD_Card_LCD.kicad_sch (KiCad schematic)
At the start: 41 parts, among them J6 Micro_SD_Card_Det1, J7 DE15_Pins_HighDensity, U3 SN74LVC2T45DCUR, U4 SN74LVC2T45DCUR, U5 TXS0102DCU

Commit message: LCD Schematic Completed
Changed lines of the file:
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@@
+	)
+	(symbol
+		(lib_id "Logsun_Logo:LOGO")
+		(at 261.62 173.99 0)
+		(unit 1)
+		(body_style 1)
+		(exclude_from_sim no)
+		(in_bom yes)
+		(on_board yes)
+		(in_pos_files yes)
+		(dnp no)
+		(fields_autoplaced yes)
+		(property "Reference" "#G8"
+			(at 261.62 168.025 0)
+			(hide yes)
+			(show_name no)
+			(do_not_autoplace no)
+			(effects
+				(font
+					(size 1.27 1.27)
+				)
+			)
+		)
+		(property "Value" "LOGO"
+			(at 261.62 179.955 0)
+			(hide yes)
+			(show_name no)
+			(do_not_autoplace no)
+			(effects
+				(font
+					(size 1.27 1.27)
+				)
+			)
+		)
+		(property "Footprint" ""
+			(at 261.62 173.99 0)
+			(hide yes)
+			(show_name no)
+			(do_not_autoplace no)
+			(effects
+				(font
+					(size 1.27 1.27)
+				)
+			)
+		)
+		(property "Datasheet" ""
+			(at 261.62 173.99 0)
+			(hide yes)
+			(show_name no)
+			(do_not_autoplace no)
+			(effects
+				(font
+					(size 1.27 1.27)
+				)
+			)
+		)
+		(property "Description" ""
+			(at 261.62 173.99 0)
+			(hide yes)
+			(show_name no)
+			(do_not_autoplace no)
+			(effects
+				(font
+					(size 1.27 1.27)
+				)
+			)
+		)
+		(instances
+			(project "DSP320C6748_DVK"
+				(path "/3a70ffc0-9fe7-4a5b-b3c2-23140355df82/5299f997-70dc-46c2-bb29-2b6cbd3c3f85"
+					(reference "#G8")
+					(unit 1)
+				)
+			)
+		)
 	)
 	(symbol

Commit message: Whole Schematic Reannotation Done
Parts:
- renumbered C103 to C100, C98 to C101, C104 to C103, C99 to C104, C101 to C105, C105 to C106, C86 to C107, C85 to C108, C95 to C89, C91 to C90, C96 to C91, C106 to C95, C107 to C96, C108 to C98, C100 to C99, D6 to D8, D7 to D9, FB6 to FB5, FB5 to FB6, J7 to J6, J6 to J7, L6 to L4, L4 to L5, L5 to L6, R106 to R86, R107 to R87, R71 to R88, R72 to R89, R73 to R90, R74 to R91, R75 to R92, R76 to R93, R77 to R94, U5 to U3, U3 to U4, U4 to U5

Commit message: DC jack Replaced With Type-C, ADC and RTC section added
Parts:
- renumbered C98 to C100, C99 to C101, C100 to C102, C101 to C103, C102 to C104, C103 to C105, C104 to C106, C105 to C107, C106 to C108, C107 to C109, C108 to C110, C89 to C91, C90 to C92, C91 to C93, C92 to C94, C93 to C95, C94 to C96, C95 to C97, C96 to C98, C97 to C99, FB5 to FB7, FB6 to FB8, J6 to J7, J7 to J8, R86 to R87, R87 to R88, R88 to R89, R89 to R90, R90 to R91, R91 to R92, R92 to R93, R93 to R94, R94 to R95

Commit message: Scheamtic Re-annotation done, Some footprints assigned
Parts:
- C100: renamed from C97; footprint (none) -> Capacitor_SMD:C_0603_1608Metric_Pad1.08x0.95mm_HandSolder
- C101: renamed from C98; footprint (none) -> Capacitor_SMD:C_0603_1608Metric_Pad1.08x0.95mm_HandSolder
- C102: renamed from C99; footprint (none) -> Capacitor_SMD:C_0603_1608Metric_Pad1.08x0.95mm_HandSolder
- C103: renamed from C100; footprint (none) -> Capacitor_SMD:C_0603_1608Metric_Pad1.08x0.95mm_HandSolder
- C104: renamed from C101; footprint (none) -> Capacitor_SMD:C_0603_1608Metric_Pad1.08x0.95mm_HandSolder
- C105: renamed from C102; footprint (none) -> Capacitor_SMD:C_0603_1608Metric_Pad1.08x0.95mm_HandSolder
- C106: renamed from C103; footprint (none) -> Capacitor_SMD:C_0603_1608Metric_Pad1.08x0.95mm_HandSolder
- C107: renamed from C104; footprint (none) -> Capacitor_SMD:C_0603_1608Metric_Pad1.08x0.95mm_HandSolder
- C108: renamed from C105; footprint (none) -> Capacitor_SMD:C_0603_1608Metric_Pad1.08x0.95mm_HandSolder
- C109: renamed from C106; footprint (none) -> Capacitor_SMD:C_0603_1608Metric_Pad1.08x0.95mm_HandSolder
- C110: renamed from C107; footprint (none) -> Capacitor_SMD:C_0603_1608Metric_Pad1.08x0.95mm_HandSolder
- C111: renamed from C108; footprint (none) -> Capacitor_SMD:C_0603_1608Metric_Pad1.08x0.95mm_HandSolder
- C112: renamed from C109; footprint (none) -> Capacitor_SMD:C_0603_1608Metric_Pad1.08x0.95mm_HandSolder
- C113: renamed from C110; footprint (none) -> Capacitor_SMD:C_0603_1608Metric_Pad1.08x0.95mm_HandSolder
- C94: renamed from C91; footprint (none) -> Capacitor_SMD:C_0603_1608Metric_Pad1.08x0.95mm_HandSolder
- C95: renamed from C92; footprint (none) -> Capacitor_SMD:C_0603_1608Metric_Pad1.08x0.95mm_HandSolder
- C96: renamed from C93; footprint (none) -> Capacitor_SMD:C_0603_1608Metric_Pad1.08x0.95mm_HandSolder
- C97: renamed from C94; footprint (none) -> Capacitor_SMD:C_0603_1608Metric_Pad1.08x0.95mm_HandSolder
- C98: renamed from C95; footprint (none) -> Capacitor_SMD:C_0603_1608Metric_Pad1.08x0.95mm_HandSolder
- C99: renamed from C96; footprint (none) -> Capacitor_SMD:C_0603_1608Metric_Pad1.08x0.95mm_HandSolder
- FB8: renamed from FB7; footprint (none) -> Inductor_SMD:L_0805_2012Metric_Pad1.05x1.20mm_HandSolder
- FB9: renamed from FB8; footprint (none) -> Inductor_SMD:L_0805_2012Metric_Pad1.05x1.20mm_HandSolder
- R89: renamed from R87; footprint (none) -> Resistor_SMD:R_0603_1608Metric_Pad0.98x0.95mm_HandSolder
- R90: renamed from R88; footprint (none) -> Resistor_SMD:R_0603_1608Metric_Pad0.98x0.95mm_HandSolder
- R91: renamed from R89; footprint (none) -> Resistor_SMD:R_0603_1608Metric_Pad0.98x0.95mm_HandSolder
- R92: renamed from R90; footprint (none) -> Resistor_SMD:R_0603_1608Metric_Pad0.98x0.95mm_HandSolder
- R93: renamed from R91; footprint (none) -> Resistor_SMD:R_0603_1608Metric_Pad0.98x0.95mm_HandSolder
- R94: renamed from R92; footprint (none) -> Resistor_SMD:R_0603_1608Metric_Pad0.98x0.95mm_HandSolder
- R95: renamed from R93; footprint (none) -> Resistor_SMD:R_0603_1608Metric_Pad0.98x0.95mm_HandSolder
- R96: renamed from R94; footprint (none) -> Resistor_SMD:R_0603_1608Metric_Pad0.98x0.95mm_HandSolder
- R97: renamed from R95; footprint (none) -> Resistor_SMD:R_0603_1608Metric_Pad0.98x0.95mm_HandSolder
