File: DSP320C6748_DVK/DSP320C6748_DVK.kicad_pcb (KiCad board)
At the start: 8 copper layers, 0 parts

Commit message: Updated Schematic exported to PDF
Parts:
- added BATTERY1: ~, LOGSUN:LGS-KC-LEADED, F.Cu at (25.1, 57.9)
- added C1: 0.22uF/6.3V X5R, Capacitor_SMD:C_0603_1608Metric_Pad1.08x0.95mm_HandSolder, F.Cu at (94.8, 72.9)
- added C10: 0.1uF/16V/X7R, Capacitor_SMD:C_0603_1608Metric_Pad1.08x0.95mm_HandSolder, F.Cu at (94.8, 95.5)
- added C100: 100pF/25V, Capacitor_SMD:C_0603_1608Metric_Pad1.08x0.95mm_HandSolder, F.Cu at (76.0, 65.9)
- added C101: 33pF/50V, Capacitor_SMD:C_0603_1608Metric_Pad1.08x0.95mm_HandSolder, F.Cu at (76.0, 68.4)
- added C102: 0.1uF/16V/X7R, Capacitor_SMD:C_0603_1608Metric_Pad1.08x0.95mm_HandSolder, F.Cu at (80.4, 50.8)
- added C103: 270pF/50V, Capacitor_SMD:C_0603_1608Metric_Pad1.08x0.95mm_HandSolder, F.Cu at (80.4, 53.3)
- added C104: 100pF/25V, Capacitor_SMD:C_0603_1608Metric_Pad1.08x0.95mm_HandSolder, F.Cu at (80.4, 55.8)
- added C105: 100pF/25V, Capacitor_SMD:C_0603_1608Metric_Pad1.08x0.95mm_HandSolder, F.Cu at (80.4, 58.3)
- added C106: 0.1uF/16V/X7R, Capacitor_SMD:C_0603_1608Metric_Pad1.08x0.95mm_HandSolder, F.Cu at (80.4, 60.8)
- added C107: 33pF/50V, Capacitor_SMD:C_0603_1608Metric_Pad1.08x0.95mm_HandSolder, F.Cu at (80.4, 63.4)
- added C108: 33pF/50V, Capacitor_SMD:C_0603_1608Metric_Pad1.08x0.95mm_HandSolder, F.Cu at (80.4, 65.9)
- added C109: 1uF/10V/X5R, Capacitor_SMD:C_0603_1608Metric_Pad1.08x0.95mm_HandSolder, F.Cu at (80.4, 68.4)
- added C11: 0.1uF/16V/X7R, Capacitor_SMD:C_0603_1608Metric_Pad1.08x0.95mm_HandSolder, F.Cu at (99.1, 72.9)
- added C110: 270pF/50V, Capacitor_SMD:C_0603_1608Metric_Pad1.08x0.95mm_HandSolder, F.Cu at (84.7, 50.8)
- added C111: 270pF/50V, Capacitor_SMD:C_0603_1608Metric_Pad1.08x0.95mm_HandSolder, F.Cu at (84.7, 53.3)
- added C112: 0.1uF/16V/X7R, Capacitor_SMD:C_0603_1608Metric_Pad1.08x0.95mm_HandSolder, F.Cu at (84.7, 55.8)
- added C113: 10uF/10V/X5R, Capacitor_SMD:C_0603_1608Metric_Pad1.08x0.95mm_HandSolder, F.Cu at (84.7, 58.3)
- added C114: 0.1uF/16V/X7R, Capacitor_SMD:C_0603_1608Metric_Pad1.08x0.95mm_HandSolder, F.Cu at (19.0, 82.0)
- added C115: 0.1uF/16V/X7R, Capacitor_SMD:C_0603_1608Metric_Pad1.08x0.95mm_HandSolder, F.Cu at (19.0, 84.5)
- added C116: 0.1uF/16V/X7R, Capacitor_SMD:C_0603_1608Metric_Pad1.08x0.95mm_HandSolder, F.Cu at (19.0, 87.0)
- added C117: 0.1uF/16V/X7R, Capacitor_SMD:C_0603_1608Metric_Pad1.08x0.95mm_HandSolder, F.Cu at (19.0, 89.5)
- added C118: 0.1uF/16V/X7R, Capacitor_SMD:C_0603_1608Metric_Pad1.08x0.95mm_HandSolder, F.Cu at (19.0, 92.0)
- added C119: 0.1uF/16V/X7R, Capacitor_SMD:C_0603_1608Metric_Pad1.08x0.95mm_HandSolder, F.Cu at (19.0, 94.5)
- added C12: 0.1uF/16V/X7R, Capacitor_SMD:C_0603_1608Metric_Pad1.08x0.95mm_HandSolder, F.Cu at (99.1, 75.4)
- added C120: 0.1uF/16V/X7R, Capacitor_SMD:C_0603_1608Metric_Pad1.08x0.95mm_HandSolder, F.Cu at (19.0, 97.0)
- added C121: 0.1uF/16V/X7R, Capacitor_SMD:C_0603_1608Metric_Pad1.08x0.95mm_HandSolder, F.Cu at (19.0, 99.5)
- added C122: 0.1uF/16V/X7R, Capacitor_SMD:C_0603_1608Metric_Pad1.08x0.95mm_HandSolder, F.Cu at (23.3, 82.0)
- added C123: 0.1uF/16V/X7R, Capacitor_SMD:C_0603_1608Metric_Pad1.08x0.95mm_HandSolder, F.Cu at (23.3, 84.5)
- added C124: 0.1uF/16V/X7R, Capacitor_SMD:C_0603_1608Metric_Pad1.08x0.95mm_HandSolder, F.Cu at (23.3, 87.0)
- added C125: 0.1uF/16V/X7R, Capacitor_SMD:C_0603_1608Metric_Pad1.08x0.95mm_HandSolder, F.Cu at (23.3, 89.5)
- added C126: 0.1uF/16V/X7R, Capacitor_SMD:C_0603_1608Metric_Pad1.08x0.95mm_HandSolder, F.Cu at (23.3, 92.0)
- added C127: 0.1uF/16V/X7R, Capacitor_SMD:C_0603_1608Metric_Pad1.08x0.95mm_HandSolder, F.Cu at (63.3, 17.9)
- added C128: 0.1uF/16V/X7R, Capacitor_SMD:C_0603_1608Metric_Pad1.08x0.95mm_HandSolder, F.Cu at (63.3, 20.4)
- added C129: 10uF/10V/X5R, Capacitor_SMD:C_0603_1608Metric_Pad1.08x0.95mm_HandSolder, F.Cu at (63.3, 22.9)
- added C13: 0.1uF/16V/X7R, Capacitor_SMD:C_0603_1608Metric_Pad1.08x0.95mm_HandSolder, F.Cu at (99.1, 77.9)
- added C130: 0.1uF/16V/X7R, Capacitor_SMD:C_0603_1608Metric_Pad1.08x0.95mm_HandSolder, F.Cu at (63.3, 25.4)
- added C131: 0.01uF/16V/X7R, Capacitor_SMD:C_0603_1608Metric_Pad1.08x0.95mm_HandSolder, F.Cu at (63.3, 27.9)
- added C132: 0.1uF/16V/X7R, Capacitor_SMD:C_0603_1608Metric_Pad1.08x0.95mm_HandSolder, F.Cu at (63.3, 30.4)
- added C133: 0.01uF/16V/X7R, Capacitor_SMD:C_0603_1608Metric_Pad1.08x0.95mm_HandSolder, F.Cu at (63.3, 32.9)
- added C134: 0.1uF/16V/X7R, Capacitor_SMD:C_0603_1608Metric_Pad1.08x0.95mm_HandSolder, F.Cu at (63.3, 35.4)
- added C135: 0.01uF/16V/X7R, Capacitor_SMD:C_0603_1608Metric_Pad1.08x0.95mm_HandSolder, F.Cu at (63.3, 37.9)
- added C136: 0.01uF/16V/X7R, Capacitor_SMD:C_0603_1608Metric_Pad1.08x0.95mm_HandSolder, F.Cu at (63.3, 40.4)
- added C137: 10uF/10V/X5R, Capacitor_SMD:C_0603_1608Metric_Pad1.08x0.95mm_HandSolder, F.Cu at (63.3, 43.0)
- added C138: 0.1uF/16V/X7R, Capacitor_SMD:C_0603_1608Metric_Pad1.08x0.95mm_HandSolder, F.Cu at (67.6, 17.9)
- added C139: 0.1uF/16V/X7R, Capacitor_SMD:C_0603_1608Metric_Pad1.08x0.95mm_HandSolder, F.Cu at (67.6, 20.4)
- added C14: 0.1uF/16V/X7R, Capacitor_SMD:C_0603_1608Metric_Pad1.08x0.95mm_HandSolder, F.Cu at (99.1, 80.4)
- added C140: 0.01uF/16V/X7R, Capacitor_SMD:C_0603_1608Metric_Pad1.08x0.95mm_HandSolder, F.Cu at (67.6, 22.9)
- added C141: 0.01uF/16V/X7R, Capacitor_SMD:C_0603_1608Metric_Pad1.08x0.95mm_HandSolder, F.Cu at (67.6, 25.4)
- added C142: 0.1uF/16V/X7R, Capacitor_SMD:C_0603_1608Metric_Pad1.08x0.95mm_HandSolder, F.Cu at (67.6, 27.9)
- added C143: 10uF/10V/X5R, Capacitor_SMD:C_0603_1608Metric_Pad1.08x0.95mm_HandSolder, F.Cu at (67.6, 30.4)
- added C144: 0.01uF/16V/X7R, Capacitor_SMD:C_0603_1608Metric_Pad1.08x0.95mm_HandSolder, F.Cu at (67.6, 32.9)
- added C145: 0.1uF/16V/X7R, Capacitor_SMD:C_0603_1608Metric_Pad1.08x0.95mm_HandSolder, F.Cu at (86.1, 100.0)
- added C146: 0.1uF/16V/X7R, Capacitor_SMD:C_0603_1608Metric_Pad1.08x0.95mm_HandSolder, F.Cu at (86.1, 102.5)
- added C147: 0.01uF/16V/X7R, Capacitor_SMD:C_0603_1608Metric_Pad1.08x0.95mm_HandSolder, F.Cu at (86.1, 105.0)
- added C148: 1uF/10V/X5R, Capacitor_SMD:C_0603_1608Metric_Pad1.08x0.95mm_HandSolder, F.Cu at (86.1, 107.5)
- added C149: 0.1uF/16V/X7R, Capacitor_SMD:C_0603_1608Metric_Pad1.08x0.95mm_HandSolder, F.Cu at (71.0, 72.9)
- added C15: 0.1uF/16V/X7R, Capacitor_SMD:C_0603_1608Metric_Pad1.08x0.95mm_HandSolder, F.Cu at (99.1, 82.9)
- added C150: 0.1uF/16V/X7R, Capacitor_SMD:C_0603_1608Metric_Pad1.08x0.95mm_HandSolder, F.Cu at (71.0, 75.4)
- added C151: 0.1uF/16V/X7R, Capacitor_SMD:C_0603_1608Metric_Pad1.08x0.95mm_HandSolder, F.Cu at (71.0, 77.9)
- added C152: 0.1uF/16V/X7R, Capacitor_SMD:C_0603_1608Metric_Pad1.08x0.95mm_HandSolder, F.Cu at (71.0, 80.4)
- added C153: 0.1uF/16V/X7R, Capacitor_SMD:C_0603_1608Metric_Pad1.08x0.95mm_HandSolder, F.Cu at (71.0, 82.9)
- added C154: 330pF/100V/X7R, Capacitor_SMD:C_0603_1608Metric_Pad1.08x0.95mm_HandSolder, F.Cu at (71.0, 85.4)
- added C155: 0.1uF/16V/X7R, Capacitor_SMD:C_0603_1608Metric_Pad1.08x0.95mm_HandSolder, F.Cu at (71.0, 87.9)
- added C156: 0.1uF/16V/X7R, Capacitor_SMD:C_0603_1608Metric_Pad1.08x0.95mm_HandSolder, F.Cu at (71.0, 90.5)
- added C157: 0.1uF/16V/X7R, Capacitor_SMD:C_0603_1608Metric_Pad1.08x0.95mm_HandSolder, F.Cu at (71.0, 93.0)
- added C158: 0.1uF/16V/X7R, Capacitor_SMD:C_0603_1608Metric_Pad1.08x0.95mm_HandSolder, F.Cu at (71.0, 95.5)
- added C159: 0.1uF/16V/X7R, Capacitor_SMD:C_0603_1608Metric_Pad1.08x0.95mm_HandSolder, F.Cu at (75.4, 72.9)
- added C16: 0.1uF/16V/X7R, Capacitor_SMD:C_0603_1608Metric_Pad1.08x0.95mm_HandSolder, F.Cu at (99.1, 85.4)
- added C160: 0.1uF/16V/X7R, Capacitor_SMD:C_0603_1608Metric_Pad1.08x0.95mm_HandSolder, F.Cu at (75.4, 75.4)
- added C161: 0.1uF/16V/X7R, Capacitor_SMD:C_0603_1608Metric_Pad1.08x0.95mm_HandSolder, F.Cu at (75.4, 77.9)
- added C162: 0.1uF/16V/X7R, Capacitor_SMD:C_0603_1608Metric_Pad1.08x0.95mm_HandSolder, F.Cu at (75.4, 80.4)
- added C163: 0.1uF/16V/X7R, Capacitor_SMD:C_0603_1608Metric_Pad1.08x0.95mm_HandSolder, F.Cu at (75.4, 82.9)
- added C164: 0.1uF/16V/X7R, Capacitor_SMD:C_0603_1608Metric_Pad1.08x0.95mm_HandSolder, F.Cu at (75.4, 85.4)
- added C165: 0.1uF/16V/X7R, Capacitor_SMD:C_0603_1608Metric_Pad1.08x0.95mm_HandSolder, F.Cu at (75.4, 87.9)
- added C166: 0.1uF/16V/X7R, Capacitor_SMD:C_0603_1608Metric_Pad1.08x0.95mm_HandSolder, F.Cu at (75.4, 90.5)
- added C167: 0.1uF/16V/X7R, Capacitor_SMD:C_0603_1608Metric_Pad1.08x0.95mm_HandSolder, F.Cu at (75.4, 93.0)
- added C168: 0.1uF/16V/X7R, Capacitor_SMD:C_0603_1608Metric_Pad1.08x0.95mm_HandSolder, F.Cu at (75.4, 95.5)
- added C169: 0.1uF/16V/X7R, Capacitor_SMD:C_0603_1608Metric_Pad1.08x0.95mm_HandSolder, F.Cu at (79.7, 72.9)
- added C17: 0.1uF/16V/X7R, Capacitor_SMD:C_0603_1608Metric_Pad1.08x0.95mm_HandSolder, F.Cu at (99.1, 87.9)
- added C170: 0.1uF/16V/X7R, Capacitor_SMD:C_0603_1608Metric_Pad1.08x0.95mm_HandSolder, F.Cu at (79.7, 75.4)
- added C171: 0.1uF/16V/X7R, Capacitor_SMD:C_0603_1608Metric_Pad1.08x0.95mm_HandSolder, F.Cu at (79.7, 77.9)
- added C172: 0.1uF/16V/X7R, Capacitor_SMD:C_0603_1608Metric_Pad1.08x0.95mm_HandSolder, F.Cu at (79.7, 80.4)
- added C173: 22pF,50V NPO, Capacitor_SMD:C_0603_1608Metric_Pad1.08x0.95mm_HandSolder, F.Cu at (79.7, 82.9)
- added C174: 22pF,50V NPO, Capacitor_SMD:C_0603_1608Metric_Pad1.08x0.95mm_HandSolder, F.Cu at (79.7, 85.4)
- added C175: 0.1uF/16V/X7R, Capacitor_SMD:C_0603_1608Metric_Pad1.08x0.95mm_HandSolder, F.Cu at (79.7, 87.9)
- added C176: 0.1uF/16V/X7R, Capacitor_SMD:C_0603_1608Metric_Pad1.08x0.95mm_HandSolder, F.Cu at (94.8, 100.0)
- added C177: 1uF/16V/X7R, Capacitor_SMD:C_0603_1608Metric_Pad1.08x0.95mm_HandSolder, F.Cu at (94.8, 102.5)
- added C178: 0.1uF/16V/X7R, Capacitor_SMD:C_0603_1608Metric_Pad1.08x0.95mm_HandSolder, F.Cu at (94.8, 105.0)
- added C179: 220pF/50V X7R, Capacitor_SMD:C_0603_1608Metric_Pad1.08x0.95mm_HandSolder, F.Cu at (94.8, 107.5)
- added C18: 0.1uF/16V/X7R, Capacitor_SMD:C_0603_1608Metric_Pad1.08x0.95mm_HandSolder, F.Cu at (99.1, 90.5)
- added C180: 0.1uF/16V/X7R, Capacitor_SMD:C_0603_1608Metric_Pad1.08x0.95mm_HandSolder, F.Cu at (94.8, 110.0)
- added C181: 220pF/50V X7R, Capacitor_SMD:C_0603_1608Metric_Pad1.08x0.95mm_HandSolder, F.Cu at (94.8, 112.5)
- added C182: 0.1uF/16V/X7R, Capacitor_SMD:C_0603_1608Metric_Pad1.08x0.95mm_HandSolder, F.Cu at (94.8, 115.0)
- added C183: 0.47uF/16V/X5R, Capacitor_SMD:C_0603_1608Metric_Pad1.08x0.95mm_HandSolder, F.Cu at (99.1, 100.0)
- added C184: 0.47uF/16V/X5R, Capacitor_SMD:C_0603_1608Metric_Pad1.08x0.95mm_HandSolder, F.Cu at (99.1, 102.5)
- added C185: 0.1uF/16V/X7R, Capacitor_SMD:C_0603_1608Metric_Pad1.08x0.95mm_HandSolder, F.Cu at (99.1, 105.0)
- added C186: 0.1uF/16V/X7R, Capacitor_SMD:C_0603_1608Metric_Pad1.08x0.95mm_HandSolder, F.Cu at (99.1, 107.5)
- added C187: 0.1uF/16V/X7R, Capacitor_SMD:C_0603_1608Metric_Pad1.08x0.95mm_HandSolder, F.Cu at (99.1, 110.0)
- added C188: 10uF/10V/X5R, Capacitor_SMD:C_0603_1608Metric_Pad1.08x0.95mm_HandSolder, F.Cu at (99.1, 112.5)
- added C189: 0.1uF/16V/X7R, Capacitor_SMD:C_0603_1608Metric_Pad1.08x0.95mm_HandSolder, F.Cu at (99.1, 115.0)
- added C19: 0.1uF/16V/X7R, Capacitor_SMD:C_0603_1608Metric_Pad1.08x0.95mm_HandSolder, F.Cu at (99.1, 93.0)
- added C190: 10uF/10V/X5R, Capacitor_SMD:C_0603_1608Metric_Pad1.08x0.95mm_HandSolder, F.Cu at (103.5, 100.0)
- added C191: 10uF/10V/X5R, Capacitor_SMD:C_0603_1608Metric_Pad1.08x0.95mm_HandSolder, F.Cu at (103.5, 102.5)
- added C192: 0.1uF/16V/X7R, Capacitor_SMD:C_0603_1608Metric_Pad1.08x0.95mm_HandSolder, F.Cu at (103.5, 105.0)
- added C193: 0.1uF/16V/X7R, Capacitor_SMD:C_0603_1608Metric_Pad1.08x0.95mm_HandSolder, F.Cu at (103.5, 107.5)
- added C194: 10uF/10V/X5R, Capacitor_SMD:C_0603_1608Metric_Pad1.08x0.95mm_HandSolder, F.Cu at (103.5, 110.0)
- added C195: 0.1uF/16V/X7R, Capacitor_SMD:C_0603_1608Metric_Pad1.08x0.95mm_HandSolder, F.Cu at (103.5, 112.5)
- added C196: 0.1uF/16V/X7R, Capacitor_SMD:C_0603_1608Metric_Pad1.08x0.95mm_HandSolder, F.Cu at (19.0, 17.9)
- added C197: 1uF/10V/X5R, Capacitor_SMD:C_0603_1608Metric_Pad1.08x0.95mm_HandSolder, F.Cu at (19.0, 20.4)
- added C198: 33pF,50V NPO, Capacitor_SMD:C_0603_1608Metric_Pad1.08x0.95mm_HandSolder, F.Cu at (19.0, 22.9)
- added C199: 33pF,50V NPO, Capacitor_SMD:C_0603_1608Metric_Pad1.08x0.95mm_HandSolder, F.Cu at (19.0, 25.4)
- added C2: 0.22uF/6.3V X5R, Capacitor_SMD:C_0603_1608Metric_Pad1.08x0.95mm_HandSolder, F.Cu at (94.8, 75.4)
- added C20: 0.1uF/16V/X7R, Capacitor_SMD:C_0603_1608Metric_Pad1.08x0.95mm_HandSolder, F.Cu at (99.1, 95.5)
- added C200: 10pF, Capacitor_SMD:C_0603_1608Metric_Pad1.08x0.95mm_HandSolder, F.Cu at (19.0, 27.9)
- added C201: 10pF, Capacitor_SMD:C_0603_1608Metric_Pad1.08x0.95mm_HandSolder, F.Cu at (19.0, 30.4)
- added C202: 0.1uF/16V/X7R, Capacitor_SMD:C_0603_1608Metric_Pad1.08x0.95mm_HandSolder, F.Cu at (19.0, 32.9)
- added C203: 10pF, Capacitor_SMD:C_0603_1608Metric_Pad1.08x0.95mm_HandSolder, F.Cu at (19.0, 35.4)
- added C204: 0.1uF/16V/X7R, Capacitor_SMD:C_0603_1608Metric_Pad1.08x0.95mm_HandSolder, F.Cu at (19.0, 37.9)
- added C205: 10pF, Capacitor_SMD:C_0603_1608Metric_Pad1.08x0.95mm_HandSolder, F.Cu at (19.0, 40.4)
- added C206: 10uF/10V/X5R, Capacitor_SMD:C_0603_1608Metric_Pad1.08x0.95mm_HandSolder, F.Cu at (19.0, 43.0)
- added C207: 0.022uF,50V, Capacitor_SMD:C_0603_1608Metric_Pad1.08x0.95mm_HandSolder, F.Cu at (23.3, 17.9)
- added C208: 12.5pF, Capacitor_SMD:C_0603_1608Metric_Pad1.08x0.95mm_HandSolder, F.Cu at (19.0, 67.4)
- added C209: 12.5pF, Capacitor_SMD:C_0603_1608Metric_Pad1.08x0.95mm_HandSolder, F.Cu at (19.0, 69.9)
- added C21: 0.1uF/16V/X7R, Capacitor_SMD:C_0603_1608Metric_Pad1.08x0.95mm_HandSolder, F.Cu at (103.5, 72.9)
- added C210: 0.1uF/16V/X7R, Capacitor_SMD:C_0603_1608Metric_Pad1.08x0.95mm_HandSolder, F.Cu at (19.0, 72.4)
- added C211: 0.1uF/16V/X7R, Capacitor_SMD:C_0603_1608Metric_Pad1.08x0.95mm_HandSolder, F.Cu at (19.0, 75.0)
- added C212: 0.1uF/16V/X7R, Capacitor_SMD:C_0603_1608Metric_Pad1.08x0.95mm_HandSolder, F.Cu at (19.0, 77.5)
- added C213: 0.1uF/16V/X7R, Capacitor_SMD:C_0603_1608Metric_Pad1.08x0.95mm_HandSolder, F.Cu at (23.3, 67.4)
- added C214: 10uF/10V/X5R, Capacitor_SMD:C_0603_1608Metric_Pad1.08x0.95mm_HandSolder, F.Cu at (23.3, 69.9)
- added C215: 0.1uF/16V/X7R, Capacitor_SMD:C_0603_1608Metric_Pad1.08x0.95mm_HandSolder, F.Cu at (23.3, 72.4)
- added C22: 0.1uF/16V/X7R, Capacitor_SMD:C_0603_1608Metric_Pad1.08x0.95mm_HandSolder, F.Cu at (103.5, 75.4)
- added C23: 0.1uF/16V/X7R, Capacitor_SMD:C_0603_1608Metric_Pad1.08x0.95mm_HandSolder, F.Cu at (103.5, 77.9)
- added C24: 10uF/10V/X5R, Capacitor_SMD:C_0603_1608Metric_Pad1.08x0.95mm_HandSolder, F.Cu at (103.5, 80.4)
- added C25: 0.1uF/16V/X7R, Capacitor_SMD:C_0603_1608Metric_Pad1.08x0.95mm_HandSolder, F.Cu at (103.5, 82.9)
- added C26: 0.1uF/16V/X7R, Capacitor_SMD:C_0603_1608Metric_Pad1.08x0.95mm_HandSolder, F.Cu at (103.5, 85.4)
- added C27: 0.1uF/16V/X7R, Capacitor_SMD:C_0603_1608Metric_Pad1.08x0.95mm_HandSolder, F.Cu at (103.5, 87.9)
- added C28: 0.1uF/16V/X7R, Capacitor_SMD:C_0603_1608Metric_Pad1.08x0.95mm_HandSolder, F.Cu at (103.5, 90.5)
- added C29: 0.1uF/16V/X7R, Capacitor_SMD:C_0603_1608Metric_Pad1.08x0.95mm_HandSolder, F.Cu at (103.5, 93.0)
- added C3: 0.1uF/16V/X7R, Capacitor_SMD:C_0603_1608Metric_Pad1.08x0.95mm_HandSolder, F.Cu at (94.8, 77.9)
- added C30: 0.1uF/16V/X7R, Capacitor_SMD:C_0603_1608Metric_Pad1.08x0.95mm_HandSolder, F.Cu at (103.5, 95.5)
- added C31: 0.1uF/16V/X7R, Capacitor_SMD:C_0603_1608Metric_Pad1.08x0.95mm_HandSolder, F.Cu at (107.8, 72.9)
- added C32: 0.1uF/16V/X7R, Capacitor_SMD:C_0603_1608Metric_Pad1.08x0.95mm_HandSolder, F.Cu at (107.8, 75.4)
- added C33: 0.1uF/16V/X7R, Capacitor_SMD:C_0603_1608Metric_Pad1.08x0.95mm_HandSolder, F.Cu at (107.8, 77.9)
- added C34: 0.1uF/16V/X7R, Capacitor_SMD:C_0603_1608Metric_Pad1.08x0.95mm_HandSolder, F.Cu at (107.8, 80.4)
- added C35: 0.1uF/16V/X7R, Capacitor_SMD:C_0603_1608Metric_Pad1.08x0.95mm_HandSolder, F.Cu at (107.8, 82.9)
- added C36: 0.1uF/16V/X7R, Capacitor_SMD:C_0603_1608Metric_Pad1.08x0.95mm_HandSolder, F.Cu at (107.8, 85.4)
- added C37: 0.1uF/16V/X7R, Capacitor_SMD:C_0603_1608Metric_Pad1.08x0.95mm_HandSolder, F.Cu at (107.8, 87.9)
- added C38: 10uF/10V/X5R, Capacitor_SMD:C_0603_1608Metric_Pad1.08x0.95mm_HandSolder, F.Cu at (107.8, 90.5)
- added C39: 0.1uF/16V/X7R, Capacitor_SMD:C_0603_1608Metric_Pad1.08x0.95mm_HandSolder, F.Cu at (107.8, 93.0)
- added C4: 0.1uF/16V/X7R, Capacitor_SMD:C_0603_1608Metric_Pad1.08x0.95mm_HandSolder, F.Cu at (94.8, 80.4)
- added C40: 0.1uF/16V/X7R, Capacitor_SMD:C_0603_1608Metric_Pad1.08x0.95mm_HandSolder, F.Cu at (107.8, 95.5)
- added C41: 0.1uF/16V/X7R, Capacitor_SMD:C_0603_1608Metric_Pad1.08x0.95mm_HandSolder, F.Cu at (112.2, 72.9)
- added C42: 10uF/10V/X5R, Capacitor_SMD:C_0603_1608Metric_Pad1.08x0.95mm_HandSolder, F.Cu at (112.2, 75.4)
- added C43: 0.1uF/16V/X7R, Capacitor_SMD:C_0603_1608Metric_Pad1.08x0.95mm_HandSolder, F.Cu at (112.2, 77.9)
- added C44: 10uF/10V/X5R, Capacitor_SMD:C_0603_1608Metric_Pad1.08x0.95mm_HandSolder, F.Cu at (112.2, 80.4)
- added C45: 10uF/10V/X5R, Capacitor_SMD:C_0603_1608Metric_Pad1.08x0.95mm_HandSolder, F.Cu at (112.2, 82.9)
- added C46: 10uF/10V/X5R, Capacitor_SMD:C_0603_1608Metric_Pad1.08x0.95mm_HandSolder, F.Cu at (112.2, 85.4)
- added C47: 0.1uF/16V/X7R, Capacitor_SMD:C_0603_1608Metric_Pad1.08x0.95mm_HandSolder, F.Cu at (101.0, 50.8)
- added C48: 22pF,50V NPO, Capacitor_SMD:C_0603_1608Metric_Pad1.08x0.95mm_HandSolder, F.Cu at (101.0, 53.3)
- added C49: 10uF/10V/X5R, Capacitor_SMD:C_0603_1608Metric_Pad1.08x0.95mm_HandSolder, F.Cu at (101.0, 55.8)
- added C5: 0.1uF/16V/X7R, Capacitor_SMD:C_0603_1608Metric_Pad1.08x0.95mm_HandSolder, F.Cu at (94.8, 82.9)
- added C50: 22pF,50V NPO, Capacitor_SMD:C_0603_1608Metric_Pad1.08x0.95mm_HandSolder, F.Cu at (101.0, 58.3)
- added C51: 0.01uF/16V/X7R, Capacitor_SMD:C_0603_1608Metric_Pad1.08x0.95mm_HandSolder, F.Cu at (71.0, 100.0)
- added C52: 0.01uF/16V/X7R, Capacitor_SMD:C_0603_1608Metric_Pad1.08x0.95mm_HandSolder, F.Cu at (71.0, 102.5)
- added C53: 0.01uF/16V/X7R, Capacitor_SMD:C_0603_1608Metric_Pad1.08x0.95mm_HandSolder, F.Cu at (71.0, 105.0)
- added C54: 0.01uF/16V/X7R, Capacitor_SMD:C_0603_1608Metric_Pad1.08x0.95mm_HandSolder, F.Cu at (71.0, 107.5)
- added C55: 10uF/10V/X5R, Capacitor_SMD:C_0603_1608Metric_Pad1.08x0.95mm_HandSolder, F.Cu at (44.3, 97.5)
- added C56: 10uF/10V/X5R, Capacitor_SMD:C_0603_1608Metric_Pad1.08x0.95mm_HandSolder, F.Cu at (44.3, 100.0)
- added C57: 0.1uF/16V/X7R, Capacitor_SMD:C_0603_1608Metric_Pad1.08x0.95mm_HandSolder, F.Cu at (44.3, 102.5)
- added C58: 0.1uF/16V/X7R, Capacitor_SMD:C_0603_1608Metric_Pad1.08x0.95mm_HandSolder, F.Cu at (44.3, 105.0)
- added C59: 10uF/10V/X5R, Capacitor_SMD:C_0603_1608Metric_Pad1.08x0.95mm_HandSolder, F.Cu at (44.3, 107.5)
- added C6: 0.1uF/16V/X7R, Capacitor_SMD:C_0603_1608Metric_Pad1.08x0.95mm_HandSolder, F.Cu at (94.8, 85.4)
- added C60: 10uF/10V/X5R, Capacitor_SMD:C_0603_1608Metric_Pad1.08x0.95mm_HandSolder, F.Cu at (44.3, 110.0)
- added C61: 0.1uF/16V/X7R, Capacitor_SMD:C_0603_1608Metric_Pad1.08x0.95mm_HandSolder, F.Cu at (44.3, 112.5)
- added C62: 0.1uF/16V/X7R, Capacitor_SMD:C_0603_1608Metric_Pad1.08x0.95mm_HandSolder, F.Cu at (44.3, 115.0)
- added C63: 10uF/10V/X5R, Capacitor_SMD:C_0603_1608Metric_Pad1.08x0.95mm_HandSolder, F.Cu at (44.3, 72.9)
- added C64: 10uF/10V/X5R, Capacitor_SMD:C_0603_1608Metric_Pad1.08x0.95mm_HandSolder, F.Cu at (44.3, 75.4)
- added C65: 10uF/10V/X5R, Capacitor_SMD:C_0603_1608Metric_Pad1.08x0.95mm_HandSolder, F.Cu at (44.3, 77.9)
- added C66: 10uF/10V/X5R, Capacitor_SMD:C_0603_1608Metric_Pad1.08x0.95mm_HandSolder, F.Cu at (44.3, 80.4)
- added C67: 10uF/10V/X5R, Capacitor_SMD:C_0603_1608Metric_Pad1.08x0.95mm_HandSolder, F.Cu at (44.3, 82.9)
- added C68: 10uF/10V/X5R, Capacitor_SMD:C_0603_1608Metric_Pad1.08x0.95mm_HandSolder, F.Cu at (44.3, 85.4)
- added C69: 10uF/10V/X5R, Capacitor_SMD:C_0603_1608Metric_Pad1.08x0.95mm_HandSolder, F.Cu at (44.3, 87.9)
- added C7: 0.1uF/16V/X7R, Capacitor_SMD:C_0603_1608Metric_Pad1.08x0.95mm_HandSolder, F.Cu at (94.8, 87.9)
- added C70: 1uF/10V/X5R, Capacitor_SMD:C_0603_1608Metric_Pad1.08x0.95mm_HandSolder, F.Cu at (44.3, 90.5)
- added C71: 1uF/10V/X5R, Capacitor_SMD:C_0603_1608Metric_Pad1.08x0.95mm_HandSolder, F.Cu at (44.3, 93.0)
- added C72: 2.2uF/6.3V/X5R, Capacitor_SMD:C_0603_1608Metric_Pad1.08x0.95mm_HandSolder, F.Cu at (48.7, 72.9)
- added C73: 10uF/10V/X5R, Capacitor_SMD:C_0603_1608Metric_Pad1.08x0.95mm_HandSolder, F.Cu at (48.7, 75.4)
- added C74: 2.2uF/6.3V/X5R, Capacitor_SMD:C_0603_1608Metric_Pad1.08x0.95mm_HandSolder, F.Cu at (48.7, 77.9)
- added C75: 10uF/10V/X5R, Capacitor_SMD:C_0603_1608Metric_Pad1.08x0.95mm_HandSolder, F.Cu at (48.7, 80.4)
- added C76: 2.2uF/6.3V/X5R, Capacitor_SMD:C_0603_1608Metric_Pad1.08x0.95mm_HandSolder, F.Cu at (48.7, 82.9)
- added C77: 0.1uF/16V/X7R, Capacitor_SMD:C_0603_1608Metric_Pad1.08x0.95mm_HandSolder, F.Cu at (44.3, 50.8)
- added C78: 0.1uF/16V/X7R, Capacitor_SMD:C_0603_1608Metric_Pad1.08x0.95mm_HandSolder, F.Cu at (44.3, 53.3)
- added C79: 0.1uF/16V/X7R, Capacitor_SMD:C_0603_1608Metric_Pad1.08x0.95mm_HandSolder, F.Cu at (44.3, 55.8)
- added C8: 0.1uF/16V/X7R, Capacitor_SMD:C_0603_1608Metric_Pad1.08x0.95mm_HandSolder, F.Cu at (94.8, 90.5)
- added C80: 10uF/10V/X5R, Capacitor_SMD:C_0603_1608Metric_Pad1.08x0.95mm_HandSolder, F.Cu at (44.3, 58.3)
- added C81: 0.1uF/16V/X7R, Capacitor_SMD:C_0603_1608Metric_Pad1.08x0.95mm_HandSolder, F.Cu at (44.3, 60.8)
- added C82: 0.1uF/16V/X7R, Capacitor_SMD:C_0603_1608Metric_Pad1.08x0.95mm_HandSolder, F.Cu at (44.3, 63.4)
- added C83: 10uF/10V/X5R, Capacitor_SMD:C_0603_1608Metric_Pad1.08x0.95mm_HandSolder, F.Cu at (44.3, 65.9)
- added C84: 0.01uF/16V/X7R, Capacitor_SMD:C_0603_1608Metric_Pad1.08x0.95mm_HandSolder, F.Cu at (44.3, 68.4)
- added C85: 0.01uF/16V/X7R, Capacitor_SMD:C_0603_1608Metric_Pad1.08x0.95mm_HandSolder, F.Cu at (48.7, 50.8)
- added C86: 10pF,50V NPO, Capacitor_SMD:C_0603_1608Metric_Pad1.08x0.95mm_HandSolder, F.Cu at (48.7, 53.3)
- added C87: 10uF/10V/X5R, Capacitor_SMD:C_0603_1608Metric_Pad1.08x0.95mm_HandSolder, F.Cu at (48.7, 55.8)
- added C88: 10uF/10V/X5R, Capacitor_SMD:C_0603_1608Metric_Pad1.08x0.95mm_HandSolder, F.Cu at (48.7, 58.3)
- added C89: 4.7uF, Capacitor_SMD:C_0603_1608Metric_Pad1.08x0.95mm_HandSolder, F.Cu at (48.7, 60.8)
- added C9: 0.1uF/16V/X7R, Capacitor_SMD:C_0603_1608Metric_Pad1.08x0.95mm_HandSolder, F.Cu at (94.8, 93.0)
- added C90: 0.1uF, Capacitor_SMD:C_0603_1608Metric_Pad1.08x0.95mm_HandSolder, F.Cu at (48.7, 63.4)
- added C91: 0.1uF/16V/X7R, Capacitor_SMD:C_0603_1608Metric_Pad1.08x0.95mm_HandSolder, F.Cu at (48.7, 65.9)
- added C92: 10uF/10V/X5R, Capacitor_SMD:C_0603_1608Metric_Pad1.08x0.95mm_HandSolder, F.Cu at (48.7, 68.4)
- added C93: 0.1uF/16V/X7R, Capacitor_SMD:C_0603_1608Metric_Pad1.08x0.95mm_HandSolder, F.Cu at (53.0, 50.8)
- added C94: 0.1uF/16V/X7R, Capacitor_SMD:C_0603_1608Metric_Pad1.08x0.95mm_HandSolder, F.Cu at (76.0, 50.8)
- added C95: 0.1uF/16V/X7R, Capacitor_SMD:C_0603_1608Metric_Pad1.08x0.95mm_HandSolder, F.Cu at (76.0, 53.3)
- added C96: 0.1uF/16V/X7R, Capacitor_SMD:C_0603_1608Metric_Pad1.08x0.95mm_HandSolder, F.Cu at (76.0, 55.8)
- added C97: 0.1uF/16V/X7R, Capacitor_SMD:C_0603_1608Metric_Pad1.08x0.95mm_HandSolder, F.Cu at (76.0, 58.3)
- added C98: 0.1uF/16V/X7R, Capacitor_SMD:C_0603_1608Metric_Pad1.08x0.95mm_HandSolder, F.Cu at (76.0, 60.8)
- added C99: 0.1uF/16V/X7R, Capacitor_SMD:C_0603_1608Metric_Pad1.08x0.95mm_HandSolder, F.Cu at (76.0, 63.4)
- added D6: SP0503BAHT, Package_TO_SOT_SMD:SOT-143, F.Cu at (69.0, 62.1)
- added D8: BAV99, Package_TO_SOT_SMD:SOT-23, F.Cu at (93.7, 62.9)
- added D9: BAV99, Package_TO_SOT_SMD:SOT-23, F.Cu at (93.7, 67.4)
- added FB1: MMZ2012S121A, Inductor_SMD:L_0805_2012Metric_Pad1.05x1.20mm_HandSolder, F.Cu at (137.3, 49.1)
- added FB10: MMZ2012S121A, Inductor_SMD:L_0805_2012Metric_Pad1.05x1.20mm_HandSolder, F.Cu at (156.2, 44.5)
- added FB11: MMZ2012S121A, Inductor_SMD:L_0805_2012Metric_Pad1.05x1.20mm_HandSolder, F.Cu at (130.4, 17.1)
- added FB12: MMZ2012S121A, Inductor_SMD:L_0805_2012Metric_Pad1.05x1.20mm_HandSolder, F.Cu at (130.4, 19.9)
- added FB13: MMZ2012S121A, Inductor_SMD:L_0805_2012Metric_Pad1.05x1.20mm_HandSolder, F.Cu at (130.4, 22.6)
- added FB14: MMZ2012S121A, Inductor_SMD:L_0805_2012Metric_Pad1.05x1.20mm_HandSolder, F.Cu at (142.3, 37.0)
- added FB15: MMZ2012S121A, Inductor_SMD:L_0805_2012Metric_Pad1.05x1.20mm_HandSolder, F.Cu at (142.3, 39.8)
- added FB16: MMZ2012S121A, Inductor_SMD:L_0805_2012Metric_Pad1.05x1.20mm_HandSolder, F.Cu at (142.3, 42.5)
- added FB17: MMZ2012S121A, Inductor_SMD:L_0805_2012Metric_Pad1.05x1.20mm_HandSolder, F.Cu at (154.4, 22.2)
- added FB18: MMZ2012S121A, Inductor_SMD:L_0805_2012Metric_Pad1.05x1.20mm_HandSolder, F.Cu at (125.3, 44.4)
- added FB19: MMZ2012S121A, Inductor_SMD:L_0805_2012Metric_Pad1.05x1.20mm_HandSolder, F.Cu at (125.3, 47.1)
- added FB2: MMZ2012S121A, Inductor_SMD:L_0805_2012Metric_Pad1.05x1.20mm_HandSolder, F.Cu at (154.4, 32.0)
- added FB3: MMZ2012S121A, Inductor_SMD:L_0805_2012Metric_Pad1.05x1.20mm_HandSolder, F.Cu at (149.2, 47.3)
- added FB4: MMZ2012S121A, Inductor_SMD:L_0805_2012Metric_Pad1.05x1.20mm_HandSolder, F.Cu at (137.3, 32.3)
- added FB5: MMZ2012S121A, Inductor_SMD:L_0805_2012Metric_Pad1.05x1.20mm_HandSolder, F.Cu at (149.2, 37.0)
- added FB6: MMZ2012S121A, Inductor_SMD:L_0805_2012Metric_Pad1.05x1.20mm_HandSolder, F.Cu at (149.2, 39.8)
- added FB7: MMZ2012S121A, Inductor_SMD:L_0805_2012Metric_Pad1.05x1.20mm_HandSolder, F.Cu at (149.2, 42.5)
- added FB8: MMZ2012S121A, Inductor_SMD:L_0805_2012Metric_Pad1.05x1.20mm_HandSolder, F.Cu at (156.2, 37.0)
- added FB9: MMZ2012S121A, Inductor_SMD:L_0805_2012Metric_Pad1.05x1.20mm_HandSolder, F.Cu at (156.2, 39.8)
- added IC7: TPS3707-33DR, TPS3707-33DR:SOIC127P600X175-8N, F.Cu at (59.4, 106.7)
- added IC8: TPS650250RHBR, TPS650250RHBR:QFN50P500X500X100-33N-D, F.Cu at (63.2, 75.3)
- added IC9: CDCM61001RHBT, TPS650250RHBR:QFN50P500X500X100-33N-D, F.Cu at (63.2, 63.4)
- added J13: RJ45_Halo_HFJ11-x2450E-LxxRL, Connector_RJ:RJ45_HALO_HFJ11-x2450E-LxxRL_Horizontal, F.Cu at (44.4, 22.0)
- added J6: USB_Type_C, LOGSUN:LGS-KC-VALCON_CSP-USC16-TR, F.Cu at (65.8, 51.6)
- added R1: 0R, 5%, 1/10W, Resistor_SMD:R_0603_1608Metric_Pad0.98x0.95mm_HandSolder, F.Cu at (112.2, 87.9)
- added R10: 4.7K,5%,1/16W, Resistor_SMD:R_0603_1608Metric_Pad0.98x0.95mm_HandSolder, F.Cu at (105.4, 55.8)
- added R100: 4.7K,5%,1/16W, Resistor_SMD:R_0603_1608Metric_Pad0.98x0.95mm_HandSolder, F.Cu at (23.3, 99.5)
- added R101: 4.7K,5%,1/16W, Resistor_SMD:R_0603_1608Metric_Pad0.98x0.95mm_HandSolder, F.Cu at (27.7, 82.0)
- added R102: 75R,5%,1/16W, Resistor_SMD:R_0603_1608Metric_Pad0.98x0.95mm_HandSolder, F.Cu at (27.7, 84.5)
- added R103: 4.7K,5%,1/16W, Resistor_SMD:R_0603_1608Metric_Pad0.98x0.95mm_HandSolder, F.Cu at (27.7, 87.0)
- added R104: 75R,5%,1/16W, Resistor_SMD:R_0603_1608Metric_Pad0.98x0.95mm_HandSolder, F.Cu at (27.7, 89.5)
- added R105: 4.7K,5%,1/16W, Resistor_SMD:R_0603_1608Metric_Pad0.98x0.95mm_HandSolder, F.Cu at (27.7, 92.0)
- added R106: 75R,5%,1/16W, Resistor_SMD:R_0603_1608Metric_Pad0.98x0.95mm_HandSolder, F.Cu at (27.7, 94.5)
- added R107: 1K,1%,1/16W, Resistor_SMD:R_0603_1608Metric_Pad0.98x0.95mm_HandSolder, F.Cu at (67.6, 35.4)
- added R108: 10R,1%,1/16W, Resistor_SMD:R_0603_1608Metric_Pad0.98x0.95mm_HandSolder, F.Cu at (67.6, 37.9)
- added R109: 22R,1%,1/16W, Resistor_SMD:R_0603_1608Metric_Pad0.98x0.95mm_HandSolder, F.Cu at (67.6, 40.4)
- added R11: 10K,1%,1/16W, Resistor_SMD:R_0603_1608Metric_Pad0.98x0.95mm_HandSolder, F.Cu at (105.4, 58.3)
- added R110: 22R,1%,1/16W, Resistor_SMD:R_0603_1608Metric_Pad0.98x0.95mm_HandSolder, F.Cu at (67.6, 43.0)
- added R111: 10R,1%,1/16W, Resistor_SMD:R_0603_1608Metric_Pad0.98x0.95mm_HandSolder, F.Cu at (72.0, 17.9)
- added R112: 10R,1%,1/16W, Resistor_SMD:R_0603_1608Metric_Pad0.98x0.95mm_HandSolder, F.Cu at (72.0, 20.4)
- added R113: 10R,1%,1/16W, Resistor_SMD:R_0603_1608Metric_Pad0.98x0.95mm_HandSolder, F.Cu at (72.0, 22.9)
- added R114: 10R,1%,1/16W, Resistor_SMD:R_0603_1608Metric_Pad0.98x0.95mm_HandSolder, F.Cu at (72.0, 25.4)
- added R115: 10R,1%,1/16W, Resistor_SMD:R_0603_1608Metric_Pad0.98x0.95mm_HandSolder, F.Cu at (72.0, 27.9)
- added R116: 10R,1%,1/16W, Resistor_SMD:R_0603_1608Metric_Pad0.98x0.95mm_HandSolder, F.Cu at (72.0, 30.4)
- added R117: 10R,1%,1/16W, Resistor_SMD:R_0603_1608Metric_Pad0.98x0.95mm_HandSolder, F.Cu at (72.0, 32.9)
- added R118: 10R,1%,1/16W, Resistor_SMD:R_0603_1608Metric_Pad0.98x0.95mm_HandSolder, F.Cu at (72.0, 35.4)
- added R119: 22R,1%,1/16W, Resistor_SMD:R_0603_1608Metric_Pad0.98x0.95mm_HandSolder, F.Cu at (72.0, 37.9)
- added R12: 10K,1%,1/16W, Resistor_SMD:R_0603_1608Metric_Pad0.98x0.95mm_HandSolder, F.Cu at (105.4, 60.8)
- added R120: 22R,1%,1/16W, Resistor_SMD:R_0603_1608Metric_Pad0.98x0.95mm_HandSolder, F.Cu at (72.0, 40.4)
- added R121: 10R,1%,1/16W, Resistor_SMD:R_0603_1608Metric_Pad0.98x0.95mm_HandSolder, F.Cu at (72.0, 43.0)
- added R122: 10R,1%,1/16W, Resistor_SMD:R_0603_1608Metric_Pad0.98x0.95mm_HandSolder, F.Cu at (76.3, 17.9)
- added R123: 10R,1%,1/16W, Resistor_SMD:R_0603_1608Metric_Pad0.98x0.95mm_HandSolder, F.Cu at (76.3, 20.4)
- added R124: 1K,1%,1/16W, Resistor_SMD:R_0603_1608Metric_Pad0.98x0.95mm_HandSolder, F.Cu at (76.3, 22.9)
- added R125: 10R,1%,1/16W, Resistor_SMD:R_0603_1608Metric_Pad0.98x0.95mm_HandSolder, F.Cu at (76.3, 25.4)
- added R126: 10R,1%,1/16W, Resistor_SMD:R_0603_1608Metric_Pad0.98x0.95mm_HandSolder, F.Cu at (76.3, 27.9)
- added R127: 10R,1%,1/16W, Resistor_SMD:R_0603_1608Metric_Pad0.98x0.95mm_HandSolder, F.Cu at (76.3, 30.4)
- added R128: 10R,1%,1/16W, Resistor_SMD:R_0603_1608Metric_Pad0.98x0.95mm_HandSolder, F.Cu at (76.3, 32.9)
- added R129: 10R,1%,1/16W, Resistor_SMD:R_0603_1608Metric_Pad0.98x0.95mm_HandSolder, F.Cu at (76.3, 35.4)
- added R13: 4.7K,5%,1/16W, Resistor_SMD:R_0603_1608Metric_Pad0.98x0.95mm_HandSolder, F.Cu at (105.4, 63.4)
- added R130: 22R,1%,1/16W, Resistor_SMD:R_0603_1608Metric_Pad0.98x0.95mm_HandSolder, F.Cu at (76.3, 37.9)
- added R131: 22R,1%,1/16W, Resistor_SMD:R_0603_1608Metric_Pad0.98x0.95mm_HandSolder, F.Cu at (76.3, 40.4)
- added R132: 22R,1%,1/16W, Resistor_SMD:R_0603_1608Metric_Pad0.98x0.95mm_HandSolder, F.Cu at (76.3, 43.0)
- added R133: 10R,1%,1/16W, Resistor_SMD:R_0603_1608Metric_Pad0.98x0.95mm_HandSolder, F.Cu at (80.7, 17.9)
- added R134: 4.7K,5%,1/16W, Resistor_SMD:R_0603_1608Metric_Pad0.98x0.95mm_HandSolder, F.Cu at (80.7, 20.4)
- added R135: 22R,1%,1/16W, Resistor_SMD:R_0603_1608Metric_Pad0.98x0.95mm_HandSolder, F.Cu at (80.7, 22.9)
- added R136: 22R,1%,1/16W, Resistor_SMD:R_0603_1608Metric_Pad0.98x0.95mm_HandSolder, F.Cu at (80.7, 25.4)
- added R137: 22R,1%,1/16W, Resistor_SMD:R_0603_1608Metric_Pad0.98x0.95mm_HandSolder, F.Cu at (80.7, 27.9)
- added R138: 22R,1%,1/16W, Resistor_SMD:R_0603_1608Metric_Pad0.98x0.95mm_HandSolder, F.Cu at (80.7, 30.4)
- added R139: 22R,1%,1/16W, Resistor_SMD:R_0603_1608Metric_Pad0.98x0.95mm_HandSolder, F.Cu at (80.7, 32.9)
- added R14: 4.7K,5%,1/16W, Resistor_SMD:R_0603_1608Metric_Pad0.98x0.95mm_HandSolder, F.Cu at (105.4, 65.9)
- added R140: 10R,1%,1/16W, Resistor_SMD:R_0603_1608Metric_Pad0.98x0.95mm_HandSolder, F.Cu at (80.7, 35.4)
- added R141: 10R,1%,1/16W, Resistor_SMD:R_0603_1608Metric_Pad0.98x0.95mm_HandSolder, F.Cu at (80.7, 37.9)
- added R142: 10R,1%,1/16W, Resistor_SMD:R_0603_1608Metric_Pad0.98x0.95mm_HandSolder, F.Cu at (80.7, 40.4)
- added R143: 10R,1%,1/16W, Resistor_SMD:R_0603_1608Metric_Pad0.98x0.95mm_HandSolder, F.Cu at (80.7, 43.0)
- added R144: 10R,1%,1/16W, Resistor_SMD:R_0603_1608Metric_Pad0.98x0.95mm_HandSolder, F.Cu at (85.0, 17.9)
- added R145: 10R,1%,1/16W, Resistor_SMD:R_0603_1608Metric_Pad0.98x0.95mm_HandSolder, F.Cu at (85.0, 20.4)
- added R146: 10R,1%,1/16W, Resistor_SMD:R_0603_1608Metric_Pad0.98x0.95mm_HandSolder, F.Cu at (85.0, 22.9)
- added R147: 10R,1%,1/16W, Resistor_SMD:R_0603_1608Metric_Pad0.98x0.95mm_HandSolder, F.Cu at (85.0, 25.4)
- added R148: 10R,1%,1/16W, Resistor_SMD:R_0603_1608Metric_Pad0.98x0.95mm_HandSolder, F.Cu at (85.0, 27.9)
- added R149: 10R,1%,1/16W, Resistor_SMD:R_0603_1608Metric_Pad0.98x0.95mm_HandSolder, F.Cu at (85.0, 30.4)
- added R15: 2.2K,5%, Resistor_SMD:R_0603_1608Metric_Pad0.98x0.95mm_HandSolder, F.Cu at (105.4, 68.4)
- added R150: 10R,1%,1/16W, Resistor_SMD:R_0603_1608Metric_Pad0.98x0.95mm_HandSolder, F.Cu at (85.0, 32.9)
- added R151: 10R,1%,1/16W, Resistor_SMD:R_0603_1608Metric_Pad0.98x0.95mm_HandSolder, F.Cu at (85.0, 35.4)
- added R152: 10R,1%,1/16W, Resistor_SMD:R_0603_1608Metric_Pad0.98x0.95mm_HandSolder, F.Cu at (85.0, 37.9)
- added R153: 10R,1%,1/16W, Resistor_SMD:R_0603_1608Metric_Pad0.98x0.95mm_HandSolder, F.Cu at (85.0, 40.4)
- added R154: 4.7K,5%,1/16W, Resistor_SMD:R_0603_1608Metric_Pad0.98x0.95mm_HandSolder, F.Cu at (86.1, 110.0)
- added R155: 4.7K,5%,1/16W, Resistor_SMD:R_0603_1608Metric_Pad0.98x0.95mm_HandSolder, F.Cu at (86.1, 112.5)
- added R156: 75R,5%,1/16W, Resistor_SMD:R_0603_1608Metric_Pad0.98x0.95mm_HandSolder, F.Cu at (79.7, 90.5)
- added R157: 4.7K,5%,1/16W, Resistor_SMD:R_0603_1608Metric_Pad0.98x0.95mm_HandSolder, F.Cu at (79.7, 93.0)
- added R158: 4.7K,5%,1/16W, Resistor_SMD:R_0603_1608Metric_Pad0.98x0.95mm_HandSolder, F.Cu at (79.7, 95.5)
- added R159: 0R,5%,1/10W, Resistor_SMD:R_0603_1608Metric_Pad0.98x0.95mm_HandSolder, F.Cu at (84.1, 72.9)
- added R16: 4.7K,5%,1/16W, Resistor_SMD:R_0603_1608Metric_Pad0.98x0.95mm_HandSolder, F.Cu at (109.7, 50.8)
- added R160: 100K,5%, Resistor_SMD:R_0603_1608Metric_Pad0.98x0.95mm_HandSolder, F.Cu at (84.1, 75.4)
- added R161: 10K,1%,1/16W, Resistor_SMD:R_0603_1608Metric_Pad0.98x0.95mm_HandSolder, F.Cu at (84.1, 77.9)
- added R162: 4.7K,5%,1/16W, Resistor_SMD:R_0603_1608Metric_Pad0.98x0.95mm_HandSolder, F.Cu at (84.1, 80.4)
- added R163: 4.7K,5%,1/16W, Resistor_SMD:R_0603_1608Metric_Pad0.98x0.95mm_HandSolder, F.Cu at (84.1, 82.9)
- added R164: 4.7K,5%,1/16W, Resistor_SMD:R_0603_1608Metric_Pad0.98x0.95mm_HandSolder, F.Cu at (84.1, 85.4)
- added R165: 4.7K,5%,1/16W, Resistor_SMD:R_0603_1608Metric_Pad0.98x0.95mm_HandSolder, F.Cu at (84.1, 87.9)
- added R166: 4.7K,5%,1/16W, Resistor_SMD:R_0603_1608Metric_Pad0.98x0.95mm_HandSolder, F.Cu at (84.1, 90.5)
- added R167: 4.7K,5%,1/16W, Resistor_SMD:R_0603_1608Metric_Pad0.98x0.95mm_HandSolder, F.Cu at (84.1, 93.0)
- added R168: 4.7K,5%,1/16W, Resistor_SMD:R_0603_1608Metric_Pad0.98x0.95mm_HandSolder, F.Cu at (84.1, 95.5)
- added R169: 4.7K,5%,1/16W, Resistor_SMD:R_0603_1608Metric_Pad0.98x0.95mm_HandSolder, F.Cu at (88.4, 72.9)
- added R17: 2.2K,5%, Resistor_SMD:R_0603_1608Metric_Pad0.98x0.95mm_HandSolder, F.Cu at (109.7, 53.3)
- added R170: 4.7K,5%,1/16W, Resistor_SMD:R_0603_1608Metric_Pad0.98x0.95mm_HandSolder, F.Cu at (88.4, 75.4)
- added R171: 4.7K,5%,1/16W, Resistor_SMD:R_0603_1608Metric_Pad0.98x0.95mm_HandSolder, F.Cu at (88.4, 77.9)
- added R172: 4.7K,5%,1/16W, Resistor_SMD:R_0603_1608Metric_Pad0.98x0.95mm_HandSolder, F.Cu at (88.4, 80.4)
- added R173: 1K,5%,1/16W, Resistor_SMD:R_0603_1608Metric_Pad0.98x0.95mm_HandSolder, F.Cu at (88.4, 82.9)
- added R174: 20K,5%,1/16W, Resistor_SMD:R_0603_1608Metric_Pad0.98x0.95mm_HandSolder, F.Cu at (88.4, 85.4)
- added R175: 0R,5%,1/10W, Resistor_SMD:R_0603_1608Metric_Pad0.98x0.95mm_HandSolder, F.Cu at (103.5, 115.0)
- added R176: 0R,5%,1/10W, Resistor_SMD:R_0603_1608Metric_Pad0.98x0.95mm_HandSolder, F.Cu at (107.8, 100.0)
- added R177: 2K,1%,1,16W, Resistor_SMD:R_0603_1608Metric_Pad0.98x0.95mm_HandSolder, F.Cu at (107.8, 102.5)
- added R178: 5.6K,1%, Resistor_SMD:R_0603_1608Metric_Pad0.98x0.95mm_HandSolder, F.Cu at (107.8, 105.0)
- added R179: 5.6K,1%, Resistor_SMD:R_0603_1608Metric_Pad0.98x0.95mm_HandSolder, F.Cu at (107.8, 107.5)
- added R18: 22R,1%,1/16W, Resistor_SMD:R_0603_1608Metric_Pad0.98x0.95mm_HandSolder, F.Cu at (109.7, 55.8)
- added R180: 2K,1%,1,16W, Resistor_SMD:R_0603_1608Metric_Pad0.98x0.95mm_HandSolder, F.Cu at (107.8, 110.0)
- added R181: 2K,1%,1,16W, Resistor_SMD:R_0603_1608Metric_Pad0.98x0.95mm_HandSolder, F.Cu at (107.8, 112.5)
- added R182: 2K,1%,1,16W, Resistor_SMD:R_0603_1608Metric_Pad0.98x0.95mm_HandSolder, F.Cu at (107.8, 115.0)
- added R183: 4.7K,5%,1/16W, Resistor_SMD:R_0603_1608Metric_Pad0.98x0.95mm_HandSolder, F.Cu at (112.2, 100.0)
- added R184: 33R,5%,1/16W, Resistor_SMD:R_0603_1608Metric_Pad0.98x0.95mm_HandSolder, F.Cu at (112.2, 102.5)
- added R185: 20K,1%,1/16W, Resistor_SMD:R_0603_1608Metric_Pad0.98x0.95mm_HandSolder, F.Cu at (112.2, 105.0)
- added R186: 20K,1%,1/16W, Resistor_SMD:R_0603_1608Metric_Pad0.98x0.95mm_HandSolder, F.Cu at (112.2, 107.5)
- added R187: 20K,5%, Resistor_SMD:R_0603_1608Metric_Pad0.98x0.95mm_HandSolder, F.Cu at (112.2, 110.0)
- added R188: 2K,1%,1,16W, Resistor_SMD:R_0603_1608Metric_Pad0.98x0.95mm_HandSolder, F.Cu at (112.2, 112.5)
- added R189: 2K,1%,1,16W, Resistor_SMD:R_0603_1608Metric_Pad0.98x0.95mm_HandSolder, F.Cu at (112.2, 115.0)
- added R19: 22R,1%,1/16W, Resistor_SMD:R_0603_1608Metric_Pad0.98x0.95mm_HandSolder, F.Cu at (109.7, 58.3)
- added R190: 1.5K,1%,1,16W, Resistor_SMD:R_0603_1608Metric_Pad0.98x0.95mm_HandSolder, F.Cu at (23.3, 20.4)
- added R191: 1.5K,1%,1,16W, Resistor_SMD:R_0603_1608Metric_Pad0.98x0.95mm_HandSolder, F.Cu at (23.3, 22.9)
- added R192: 4.7K,5%,1/16W, Resistor_SMD:R_0603_1608Metric_Pad0.98x0.95mm_HandSolder, F.Cu at (23.3, 25.4)
- added R193: 100R,1%,1,16W, Resistor_SMD:R_0603_1608Metric_Pad0.98x0.95mm_HandSolder, F.Cu at (23.3, 27.9)
- added R194: 4.7K,5%,1/16W, Resistor_SMD:R_0603_1608Metric_Pad0.98x0.95mm_HandSolder, F.Cu at (23.3, 30.4)
- added R195: 100R,1%,1,16W, Resistor_SMD:R_0603_1608Metric_Pad0.98x0.95mm_HandSolder, F.Cu at (23.3, 32.9)
- added R196: 100R,1%,1,16W, Resistor_SMD:R_0603_1608Metric_Pad0.98x0.95mm_HandSolder, F.Cu at (23.3, 35.4)
- added R197: 100R,1%,1,16W, Resistor_SMD:R_0603_1608Metric_Pad0.98x0.95mm_HandSolder, F.Cu at (23.3, 37.9)
- added R198: 100R,1%,1,16W, Resistor_SMD:R_0603_1608Metric_Pad0.98x0.95mm_HandSolder, F.Cu at (23.3, 40.4)
- added R199: 100R,1%,1,16W, Resistor_SMD:R_0603_1608Metric_Pad0.98x0.95mm_HandSolder, F.Cu at (23.3, 43.0)
- added R2: 0R, Resistor_SMD:R_0603_1608Metric_Pad0.98x0.95mm_HandSolder, F.Cu at (112.2, 90.5)
- added R20: 22R,1%,1/16W, Resistor_SMD:R_0603_1608Metric_Pad0.98x0.95mm_HandSolder, F.Cu at (109.7, 60.8)
- added R200: 100R,1%,1,16W, Resistor_SMD:R_0603_1608Metric_Pad0.98x0.95mm_HandSolder, F.Cu at (27.7, 17.9)
- added R201: 100R,1%,1,16W, Resistor_SMD:R_0603_1608Metric_Pad0.98x0.95mm_HandSolder, F.Cu at (27.7, 20.4)
- added R202: 100R,1%,1,16W, Resistor_SMD:R_0603_1608Metric_Pad0.98x0.95mm_HandSolder, F.Cu at (27.7, 22.9)
- added R203: 100R,1%,1,16W, Resistor_SMD:R_0603_1608Metric_Pad0.98x0.95mm_HandSolder, F.Cu at (27.7, 25.4)
- added R204: 4.7K,5%,1/16W, Resistor_SMD:R_0603_1608Metric_Pad0.98x0.95mm_HandSolder, F.Cu at (27.7, 27.9)
- added R205: 4.7K,5%,1/16W, Resistor_SMD:R_0603_1608Metric_Pad0.98x0.95mm_HandSolder, F.Cu at (27.7, 30.4)
- added R206: 1M,1%,1/16%, Resistor_SMD:R_0603_1608Metric_Pad0.98x0.95mm_HandSolder, F.Cu at (27.7, 32.9)
- added R207: 4.7K,5%,1/16W, Resistor_SMD:R_0603_1608Metric_Pad0.98x0.95mm_HandSolder, F.Cu at (27.7, 35.4)
- added R208: 10R,1%,1/16W, Resistor_SMD:R_0603_1608Metric_Pad0.98x0.95mm_HandSolder, F.Cu at (27.7, 37.9)
- added R209: 4.7K,5%,1/16W, Resistor_SMD:R_0603_1608Metric_Pad0.98x0.95mm_HandSolder, F.Cu at (27.7, 40.4)
- added R21: 100R,1%,1/16W, Resistor_SMD:R_0603_1608Metric_Pad0.98x0.95mm_HandSolder, F.Cu at (109.7, 63.4)
- added R210: 4.7K,5%,1/16W, Resistor_SMD:R_0603_1608Metric_Pad0.98x0.95mm_HandSolder, F.Cu at (27.7, 43.0)
- added R211: 12.1K,1%,1,16W, Resistor_SMD:R_0603_1608Metric_Pad0.98x0.95mm_HandSolder, F.Cu at (32.0, 17.9)
- added R212: 4.7K,5%,1/16W, Resistor_SMD:R_0603_1608Metric_Pad0.98x0.95mm_HandSolder, F.Cu at (32.0, 20.4)
- added R213: 4.7K,5%,1/16W, Resistor_SMD:R_0603_1608Metric_Pad0.98x0.95mm_HandSolder, F.Cu at (32.0, 22.9)
- added R214: 0R,5%,1/10W, Resistor_SMD:R_0603_1608Metric_Pad0.98x0.95mm_HandSolder, F.Cu at (32.0, 25.4)
- added R215: 49.9R,1%,1/16W, Resistor_SMD:R_0603_1608Metric_Pad0.98x0.95mm_HandSolder, F.Cu at (32.0, 27.9)
- added R216: 49.9R,1%,1/16W, Resistor_SMD:R_0603_1608Metric_Pad0.98x0.95mm_HandSolder, F.Cu at (32.0, 30.4)
- added R217: 0R,5%,1/10W, Resistor_SMD:R_0603_1608Metric_Pad0.98x0.95mm_HandSolder, F.Cu at (32.0, 32.9)
- added R218: 0R,5%,1/10W, Resistor_SMD:R_0603_1608Metric_Pad0.98x0.95mm_HandSolder, F.Cu at (32.0, 35.4)
- added R219: 0R,5%,1/10W, Resistor_SMD:R_0603_1608Metric_Pad0.98x0.95mm_HandSolder, F.Cu at (32.0, 37.9)
- added R22: 10K,1%,1/16W, Resistor_SMD:R_0603_1608Metric_Pad0.98x0.95mm_HandSolder, F.Cu at (109.7, 65.9)
- added R220: 0R,5%,1/10W, Resistor_SMD:R_0603_1608Metric_Pad0.98x0.95mm_HandSolder, F.Cu at (32.0, 40.4)
- added R221: 0R,5%,1/10W, Resistor_SMD:R_0603_1608Metric_Pad0.98x0.95mm_HandSolder, F.Cu at (32.0, 43.0)
- added R222: 0R,5%,1/10W, Resistor_SMD:R_0603_1608Metric_Pad0.98x0.95mm_HandSolder, F.Cu at (36.4, 17.9)
- added R223: 49.9R,1%,1/16W, Resistor_SMD:R_0603_1608Metric_Pad0.98x0.95mm_HandSolder, F.Cu at (36.4, 20.4)
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